File: Cellule_de_force_V2.kicad_pcb (KiCad board)
At the start: 6 copper layers, 0 parts

Commit message: [PCB fini]
Parts:
- added C1: 0.1µF, Capacitor_SMD:C_0603_1608Metric, F.Cu at (190.4, 117.4)
- added C10: 0.01µF, Capacitor_SMD:C_0603_1608Metric, F.Cu at (153.2, 82.3)
- added C11: 22pf, Capacitor_SMD:C_0603_1608Metric, F.Cu at (146.8, 94.7)
- added C12: 22pf, Capacitor_SMD:C_0603_1608Metric, F.Cu at (143.7, 94.7)
- added C13: 4.7µF, Capacitor_SMD:C_0603_1608Metric, F.Cu at (198.3, 92.7)
- added C14: TAJA225K016RNJ, TAJA225K016RNJ:CAPPM3216X180N, F.Cu at (203.3, 97.8)
- added C15: 10µF, Capacitor_SMD:C_0603_1608Metric, F.Cu at (198.3, 95.2)
- added C16: 4.7µF, Capacitor_SMD:C_0603_1608Metric, F.Cu at (198.3, 97.8)
- added C17: 2.2nF, Capacitor_SMD:C_0603_1608Metric, F.Cu at (151.8, 127.8)
- added C18: 100nF, Capacitor_SMD:C_0603_1608Metric, F.Cu at (153.3, 127.8)
- added C19: 10µF, Capacitor_SMD:C_0603_1608Metric, F.Cu at (142.1, 133.6)
- added C2: 10µF, Capacitor_SMD:C_0603_1608Metric, F.Cu at (190.4, 119.9)
- added C20: 10µF, Capacitor_SMD:C_0603_1608Metric, F.Cu at (140.6, 133.6)
- added C21: 10µF, Capacitor_SMD:C_0603_1608Metric, F.Cu at (153.3, 130.8)
- added C22: 1µF, Capacitor_SMD:C_0603_1608Metric, F.Cu at (151.8, 130.8)
- added C3: 0.1µF, Capacitor_SMD:C_0603_1608Metric, F.Cu at (190.4, 122.4)
- added C4: 10µF, Capacitor_SMD:C_0603_1608Metric, F.Cu at (190.4, 124.9)
- added C5: 0.1µF, Capacitor_SMD:C_0603_1608Metric, F.Cu at (145.4, 83.8)
- added C6: 0.1µF, Capacitor_SMD:C_0603_1608Metric, F.Cu at (151.6, 83.8)
- added C7: 0.01µF, Capacitor_SMD:C_0603_1608Metric, F.Cu at (147.0, 82.3)
- added C8: 0.01µF, Capacitor_SMD:C_0603_1608Metric, F.Cu at (150.0, 82.3)
- added C9: 0.01µF, Capacitor_SMD:C_0603_1608Metric, F.Cu at (143.8, 82.3)
- added D1: LED, LED_SMD:LED_0603_1608Metric, F.Cu at (160.5, 89.8)
- added D2: LED, LED_SMD:LED_0603_1608Metric, F.Cu at (160.5, 91.3)
- added D3: PMEG2010AEH, Diode_SMD:D_SOD-123F, F.Cu at (143.9, 136.3)
- added D4: LED, LED_SMD:LED_0603_1608Metric, F.Cu at (202.4, 100.7)
- added FID1: Fiducial, Fiducial:Fiducial_1.5mm_Mask3mm, F.Cu at (279.2, 24.4)
- added FID2: Fiducial, Fiducial:Fiducial_1.5mm_Mask3mm, F.Cu at (279.2, 29.0)
- added FID3: Fiducial, Fiducial:Fiducial_1.5mm_Mask3mm, F.Cu at (283.7, 24.4)
- added FID4: Fiducial, Fiducial:Fiducial_1.5mm_Mask3mm, F.Cu at (283.7, 29.0)
- added FID5: Fiducial, Fiducial:Fiducial_1.5mm_Mask3mm, F.Cu at (288.3, 24.4)
- added FID6: Fiducial, Fiducial:Fiducial_1.5mm_Mask3mm, F.Cu at (288.3, 29.0)
- added H1: MountingHole_Pad, MountingHole:MountingHole_3.2mm_M3_Pad_Via, F.Cu at (158.5, 78.8)
- added H2: MountingHole_Pad, MountingHole:MountingHole_3.2mm_M3_Pad_Via, F.Cu at (138.6, 78.8)
- added H3: MountingHole_Pad, MountingHole:MountingHole_3.2mm_M3_Pad_Via, F.Cu at (138.6, 139.9)
- added H4: MountingHole_Pad, MountingHole:MountingHole_3.2mm_M3_Pad_Via, F.Cu at (158.5, 139.9)
- added IC2: TPS61086DRCR, TPS61086DRCR:TPS16412DRCR, F.Cu at (148.3, 129.6)
- added J1: Conn_01x02_Pin, Connector_PinHeader_2.54mm:PinHeader_1x02_P2.54mm_Vertical, F.Cu at (271.3, 58.2)
- added J2: Conn_01x02_Pin, Connector_PinHeader_2.54mm:PinHeader_1x02_P2.54mm_Vertical, F.Cu at (275.8, 58.2)
- added J3: Conn_01x02_Pin, Connector_PinHeader_2.54mm:PinHeader_1x02_P2.54mm_Vertical, F.Cu at (280.4, 58.2)
- added J4: Conn_01x02_Pin, Connector_PinHeader_2.54mm:PinHeader_1x02_P2.54mm_Vertical, F.Cu at (285.0, 58.2)
- added J5: Conn_01x04_Socket, Connector_PinSocket_2.54mm:PinSocket_1x04_P2.54mm_Vertical, F.Cu at (144.7, 76.6)
- added J6: Conn_01x05_Pin, Connector_PinSocket_2.54mm:PinSocket_1x05_P2.54mm_Vertical, F.Cu at (136.2, 84.0)
- added L1: 7447785004, 7447785004:7447785004, F.Cu at (150.3, 136.3)
- added R1: 100Ω, Resistor_SMD:R_0603_1608Metric, F.Cu at (152.4, 80.0)
- added R10: 100Ω, Resistor_SMD:R_0603_1608Metric, F.Cu at (157.5, 89.8)
- added R11: 100Ω, Resistor_SMD:R_0603_1608Metric, F.Cu at (157.5, 91.3)
- added R12: 715kΩ, Resistor_SMD:R_0603_1608Metric, F.Cu at (198.3, 102.8)
- added R13: 50kΩ, Resistor_SMD:R_0603_1608Metric, F.Cu at (198.3, 105.3)
- added R14: 200kΩ, Resistor_SMD:R_0603_1608Metric, F.Cu at (198.3, 107.8)
- added R15: 18kΩ, Resistor_SMD:R_0603_1608Metric, F.Cu at (148.0, 126.1)
- added R16: 620Ω, Resistor_SMD:R_0603_1608Metric, F.Cu at (198.3, 110.3)
- added R17: 69.8kΩ, Resistor_SMD:R_0603_1608Metric, F.Cu at (148.0, 124.6)
- added R18: 37.4kΩ, Resistor_SMD:R_0603_1608Metric, F.Cu at (151.0, 125.6)
- added R2: 100Ω, Resistor_SMD:R_0603_1608Metric, F.Cu at (150.8, 80.0)
- added R3: 100Ω, Resistor_SMD:R_0603_1608Metric, F.Cu at (139.5, 89.2)
- added R4: 100Ω, Resistor_SMD:R_0603_1608Metric, F.Cu at (139.5, 84.0)
- added R5: 100Ω, Resistor_SMD:R_0603_1608Metric, F.Cu at (139.5, 91.7)
- added R6: 100Ω, Resistor_SMD:R_0603_1608Metric, F.Cu at (139.5, 94.1)
- added R7: 100Ω, Resistor_SMD:R_0603_1608Metric, F.Cu at (139.5, 86.6)
- added R8: 100kΩ, Resistor_SMD:R_0603_1608Metric, F.Cu at (143.3, 90.0)
- added R9: 50kΩ, Resistor_SMD:R_0603_1608Metric, F.Cu at (198.3, 100.3)
- added TP1: TestPoint, TestPoint:TestPoint_Pad_D2.0mm, F.Cu at (176.0, 85.4)
- added TP14: TestPoint, TestPoint:TestPoint_Pad_D2.0mm, F.Cu at (142.7, 105.7)
- added TP15: TestPoint, TestPoint:TestPoint_Pad_D2.0mm, F.Cu at (147.8, 105.7)
- added TP16: TestPoint, TestPoint:TestPoint_Pad_D2.0mm, F.Cu at (194.3, 97.6)
- added TP17: TestPoint, TestPoint:TestPoint_Pad_D2.0mm, F.Cu at (194.3, 101.6)
- added TP18: TestPoint, TestPoint:TestPoint_Pad_D2.0mm, F.Cu at (194.3, 105.7)
- added TP19: TestPoint, TestPoint:TestPoint_Pad_D2.0mm, F.Cu at (298.6, 56.2)
- added TP2: TestPoint, TestPoint:TestPoint_Pad_D2.0mm, F.Cu at (176.0, 89.5)
- added TP20: TestPoint, TestPoint:TestPoint_Pad_D2.0mm, F.Cu at (298.6, 60.2)
- added TP21: TestPoint, TestPoint:TestPoint_Pad_D2.0mm, F.Cu at (298.6, 64.3)
- added TP22: TestPoint, TestPoint:TestPoint_Pad_D2.0mm, F.Cu at (298.6, 68.3)
- added TP23: TestPoint, TestPoint:TestPoint_Pad_D2.0mm, F.Cu at (194.3, 109.7)
- added TP3: TestPoint, TestPoint:TestPoint_Pad_D2.0mm, F.Cu at (176.0, 93.5)
- added TP4: TestPoint, TestPoint:TestPoint_Pad_D2.0mm, F.Cu at (176.0, 97.5)
- added TP5: TestPoint, TestPoint:TestPoint_Pad_D2.0mm, F.Cu at (176.0, 101.6)
- added TP6: TestPoint, TestPoint:TestPoint_Pad_D2.0mm, F.Cu at (156.3, 134.0)
- added TP7: TestPoint, TestPoint:TestPoint_Pad_D2.0mm, F.Cu at (180.1, 89.5)
- added TP8: TestPoint, TestPoint:TestPoint_Pad_D2.0mm, F.Cu at (194.3, 93.5)
- added U1: AD7190WBRUZ, AD7190WBRUZ:SOP65P640X120-24N, F.Cu at (148.5, 90.0)
- added U2: LT3042IMSE, Package_SO:MSOP-10-1EP_3x3mm_P0.5mm_EP2.2x3.1mm_Mask1.83x1.89mm_ThermalVias, F.Cu at (148.4, 115.6)
- added Y1: ABC2-4.9152MHZ-4-T, ABC2-4.9152MHZ-4-T:ABC210000MHZ4, F.Cu at (145.3, 99.8)
Routing:
- net IN-SENSE+: track 0.00 -> 19.9 mm, vias 0 -> 2
- net IN-SENSE-: track 0.00 -> 15.0 mm
- net MCLK1: track 0.00 -> 14.6 mm
- net MCLK2: track 0.00 -> 14.5 mm
- net OUT-: track 0.00 -> 12.2 mm
- net Net-(U1-P3): track 0.00 -> 11.0 mm
- net Net-(U1-~{CS}): track 0.00 -> 10.9 mm, vias 0 -> 2
- net Net-(U1-P2): track 0.00 -> 9.71 mm
- net Net-(U1-~{SYNC}): track 0.00 -> 7.76 mm
- net Net-(U1-SCLK): track 0.00 -> 6.98 mm
- net Net-(U1-DOUT/~{RDY}): track 0.00 -> 6.47 mm
- net OUT+: track 0.00 -> 6.43 mm
- net Net-(U1-DIN): track 0.00 -> 5.47 mm
- net +3.3V_IN: track 0.00 -> 5.09 mm
- net IN-OUT-: track 0.00 -> 2.99 mm
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Other:
- board outline added: 26.9 x 68.1 mm
- copper layers 6 -> 2
