File: Cellule_de_force_V2.kicad_pcb (KiCad board)
At the start: 2 copper layers, 26.9 x 68.1 mm, 83 parts, among them IC2 TPS61086DRCR, J1 Conn_01x02_Pin, J2 Conn_01x02_Pin, J3 Conn_01x02_Pin, J4 Conn_01x02_Pin, J5 Conn_01x04_Socket, J6 Conn_01x05_Pin, U1 AD7190WBRUZ, U2 LT3042IMSE, Y1 ABC2-4.9152MHZ-4-T

Commit message: [PCB 2]
Parts:
- removed FID1, FID2, FID3, FID4, FID5, FID6: Fiducial, Fiducial:Fiducial_1.5mm_Mask3mm
- removed TP1, TP2, TP21, TP22, TP23, TP5, TP7: TestPoint, TestPoint:TestPoint_Pad_D2.0mm
- moved TP20 175.5 mm to (139.4, 134.1)
- moved TP19 161.9 mm to (150.8, 122.2)
- moved J2 149.6 mm to (140.1, 121.2), turned to 180 degrees
- moved J4 132.4 mm to (158.9, 98.6)
- moved J1 132.1 mm to (160.2, 129.8), turned to 180 degrees
- moved J3 131.5 mm to (155.3, 98.6)
- moved R14 52.9 mm to (145.8, 114.2), turned to -90 degrees
- moved TP16 52.3 mm to (143.8, 111.2)
- moved C16 52.1 mm to (148.2, 111.9)
- moved C3 51.6 mm to (153.5, 86.3), turned to -90 degrees
- moved C14 51.3 mm to (154.0, 112.0), turned to 90 degrees
- moved C4 51.3 mm to (153.5, 89.3), turned to 90 degrees
- moved C13 50.9 mm to (151.2, 112.0), turned to 180 degrees
- moved C15 49.6 mm to (151.2, 110.5), turned to 180 degrees
- moved R12 48.3 mm to (152.2, 117.4), turned to -90 degrees
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Routing:
- net +5VA_OUT: track 0.00 -> 10.6 mm, vias 0 -> 2
- net IN-SENSE+: track 19.9 -> 27.8 mm
- net OUT-: track 12.2 -> 18.4 mm, vias 0 -> 2
- net OUT+: track 6.43 -> 11.5 mm
- net +6V_IN: track 0.00 -> 4.83 mm
- net /Project Architecture/LT3042_6V_5VA/PGFB: track 0.00 -> 2.73 mm
- net Net-(U2-PG): track 0.00 -> 1.76 mm
Other:
- board text removed: "Bottom View"
- board text removed: "Top View"
