File: Cellule_de_force_V2.kicad_pcb (KiCad board)
At the start: 2 copper layers, 26.9 x 68.1 mm, 70 parts, among them IC2 TPS61086DRCR, J1 Conn_01x02_Pin, J2 Conn_01x02_Pin, J3 Conn_01x02_Pin, J4 Conn_01x02_Pin, J5 Conn_01x04_Socket, J6 Conn_01x05_Pin, U1 AD7190WBRUZ, U2 LT3042IMSE, Y1 ABC2-4.9152MHZ-4-T

Commit message: [PCB 4 layer]
Parts:
- removed J2, J4: Conn_01x02_Pin, Connector_PinHeader_2.54mm:PinHeader_1x02_P2.54mm_Vertical
- removed J5: Conn_01x04_Socket, Connector_PinSocket_2.54mm:PinSocket_1x04_P2.54mm_Vertical
- removed J6: Conn_01x05_Pin, Connector_PinSocket_2.54mm:PinSocket_1x05_P2.54mm_Vertical
- removed R4, R5, R7: 100Ω, Resistor_SMD:R_0603_1608Metric
- removed TP14, TP15, TP16, TP17, TP18, TP19, TP20, TP3, TP4, TP6, TP8: TestPoint, TestPoint:TestPoint_Pad_D2.0mm
- removed Y1: ABC2-4.9152MHZ-4-T, ABC2-4.9152MHZ-4-T:ABC210000MHZ4
- added C23: 0.1µF, Capacitor_SMD:C_0603_1608Metric, F.Cu at (157.0, 86.7)
- added C24: 18pf, Capacitor_SMD:C_0603_1608Metric, F.Cu at (153.9, 93.7)
- added C25: 18pf, Capacitor_SMD:C_0603_1608Metric, F.Cu at (153.9, 96.7)
- added C26: 0.1µF, Capacitor_SMD:C_0603_1608Metric, F.Cu at (157.0, 91.2)
- added H5: WE-SHC_THT-FRAME, WE-SHC_THT-FRAME:WE-SHC_THT-FRAME_36503205, F.Cu at (148.5, 90.0)
- added Q1: SI2303CDS-T1-GE3, Package_TO_SOT_SMD:SOT-23-3, F.Cu at (153.8, 88.4)
- added RN1: RP_100Ω, Resistor_SMD:R_Array_Concave_4x0603, F.Cu at (148.5, 105.6)
- added Y2: CSTCR4M91G53-R0, CSTCR4M91G53-R0:OSC_CSTCR4M91G53-R0, F.Cu at (156.2, 95.1)
- C11: value 22pf -> 0.1µF
- C12: value 22pf -> 10µF
- D2: value LED -> RED
- J1: value Conn_01x02_Pin -> Conn_01x07_Pin; footprint Connector_PinHeader_2.54mm:PinHeader_1x02_P2.54mm_Vertical -> Connector_JST:JST_XH_B7B-XH-AM_1x07_P2.50mm_Vertical
- J3: value Conn_01x02_Pin -> 691408720004B; footprint Connector_PinHeader_2.54mm:PinHeader_1x02_P2.54mm_Vertical -> 691408720004B:691408720004B
- R10: value 100Ω -> 1kΩ
- moved C20 47.0 mm to (169.5, 95.1), turned to 0 degrees
- moved D3 45.4 mm to (166.9, 97.1), turned to -90 degrees
- moved C19 44.9 mm to (169.5, 96.6), turned to 0 degrees
- moved R17 37.2 mm to (175.7, 99.8), turned to 90 degrees
- moved R15 37.1 mm to (174.2, 99.8), turned to -90 degrees
- moved IC2 37.0 mm to (170.8, 100.1), turned to 180 degrees
- moved R12 36.7 mm to (173.8, 87.7)
- moved L1 35.6 mm to (164.1, 103.5), turned to 180 degrees
- moved R13 35.1 mm to (172.3, 87.7)
- moved R9 34.9 mm to (172.8, 85.5)
- moved R18 33.6 mm to (175.7, 102.9), turned to 90 degrees
- moved C17 32.5 mm to (173.5, 103.6), turned to 180 degrees
- moved C22 32.4 mm to (169.6, 103.7), turned to 0 degrees
- moved H3 32.2 mm to (123.5, 111.5)
- moved H4 32.1 mm to (173.5, 111.5)
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Connections:
- net Net-(U1-P3) renamed P3
- C1 pad 1: +3.3V_IN -> +3.3V
- C11 pad 1: MCLK2 -> SENSE+
- C12 pad 1: MCLK1 -> +5VA
- C13 pad 1: +5VA_OUT -> +5VA
- C15 pad 1: +5VA_OUT -> +5VA
- C16 pad 1: +6V_IN -> +6V
- C19 pad 1: +6V_OUT -> +6V
- C2 pad 1: +3.3V_IN -> +3.3V
- C20 pad 1: +6V_OUT -> +6V
- C21 pad 1: +3.3V_IN -> +3.3V
- C22 pad 1: +3.3V_IN -> +3.3V
- C3 pad 2: IN-SENSE+ -> +5VA
- C4 pad 2: IN-SENSE+ -> +5VA
- C5 pad 1: IN-SENSE+ -> SENSE+
- C5 pad 2: IN-SENSE- -> SENSE-
- C7 pad 2: IN-SENSE+ -> SENSE+
- C9 pad 1: IN-SENSE- -> SENSE-
- D3 pad 1: +6V_OUT -> +6V
- IC2 pad 3: +3.3V_IN -> +3.3V
- IC2 pad 8: +3.3V_IN -> +3.3V
- J1 pad 1: +3.3V_IN -> GND
- J1 pad 2: GND -> DOUT
- J3 pad 1: +3.3V_IN -> SENSE-
- J3 pad 2: +3.3V_IN -> SENSE+
- L1 pad 1: +3.3V_IN -> +3.3V
- R10 pad 2: Net-(D1-A) -> Net-(Q1-G)
- R12 pad 2: +5VA_OUT -> +5VA
- R14 pad 1: +6V_IN -> +6V
- R16 pad 2: +5VA_OUT -> +5VA
- R17 pad 2: +6V_OUT -> +6V
- R3 pad 1: DIN -> Net-(D1-A)
- R3 pad 2: Net-(U1-DIN) -> +3.3V
- R8 pad 1: +3.3V_IN -> +3.3V
- U1 pad 15: IN-SENSE+ -> SENSE+
- U1 pad 16: IN-SENSE- -> SENSE-
- U1 pad 20: IN-SENSE+ -> +5VA
- U1 pad 21: +3.3V_IN -> +3.3V
- U1 pad 24: Net-(U1-DIN) -> Net-(RN1-R4.1)
- U1 pad 9: (no net) -> GND
- U2 pad 1: +6V_IN -> +6V
- U2 pad 10: +5VA_OUT -> +5VA
- U2 pad 2: +6V_IN -> +6V
- U2 pad 3: +6V_IN -> +6V
- U2 pad 9: +5VA_OUT -> +5VA
Routing:
- net GND: track 0.02 -> 46.4 mm, vias 0 -> 12
- net +3.3V: track 0.00 -> 42.4 mm, vias 0 -> 3
- net IN-SENSE+: track 27.8 -> 0.00 mm, vias 2 -> 0
- net Net-(U1-P2): track 9.71 -> 33.1 mm, vias 0 -> 2
- net SENSE-: track 0.00 -> 23.0 mm
- net SENSE+: track 0.00 -> 20.1 mm, vias 0 -> 16
- net IN-SENSE-: track 15.0 -> 0.00 mm
- net +5VA: track 0.00 -> 13.3 mm, vias 0 -> 16
- net Net-(RN1-R4.1): track 0.00 -> 11.1 mm
- net +5VA_OUT: track 10.6 -> 0.00 mm, vias 2 -> 0
- net +6V: track 0.00 -> 9.50 mm, vias 0 -> 2
- net MCLK2: track 14.5 -> 6.13 mm
- net OUT-: track 18.4 -> 10.8 mm, vias 2 -> 0
- net MCLK1: track 14.6 -> 7.07 mm
- net P3: track 11.0 -> 4.04 mm
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- added copper zone on F.Cu, net +3.3V
- added copper zone on F.Cu, net +5VA
- added copper zone on In2.Cu, net +5VA
- added copper zone on F.Cu, net +6V
- added copper zone on B.Cu, net GND
- added copper zone on F.Cu, net GND
- added copper zone on In1.Cu, net GND
- added copper zone on F.Cu, net Net-(D3-A)
- added copper zone on F.Cu, net SENSE+
- added copper zone on In2.Cu, net SENSE+
Other:
- board size 26.9 x 68.1 mm -> 57 x 50.8 mm
- copper layers 2 -> 4

Commit message: [PCB V1]
Parts:
- added FID1: Fiducial, Fiducial:Fiducial_1.5mm_Mask3mm, F.Cu at (206.0, 79.8)
- added FID2: Fiducial, Fiducial:Fiducial_1.5mm_Mask3mm, F.Cu at (206.0, 84.4)
- added FID3: Fiducial, Fiducial:Fiducial_1.5mm_Mask3mm, F.Cu at (210.5, 79.8)
- added FID4: Fiducial, Fiducial:Fiducial_1.5mm_Mask3mm, F.Cu at (210.5, 84.4)
- added FID5: Fiducial, Fiducial:Fiducial_1.5mm_Mask3mm, F.Cu at (215.1, 79.8)
- added FID6: Fiducial, Fiducial:Fiducial_1.5mm_Mask3mm, F.Cu at (215.1, 84.4)
- moved R17 49.2 mm to (127.2, 91.5), turned to 180 degrees
- moved R15 47.5 mm to (127.2, 93.0), turned to 0 degrees
- moved C19 46.4 mm to (123.3, 92.5), turned to 180 degrees
- moved C20 46.2 mm to (123.3, 94.0), turned to 180 degrees
- moved R18 45.6 mm to (131.1, 93.9), turned to -90 degrees
- moved C17 45.4 mm to (129.6, 92.2), turned to 90 degrees
- moved IC2 43.4 mm to (127.5, 96.5), turned to -90 degrees
- moved D3 43.2 mm to (123.7, 97.0)
- moved R14 42.7 mm to (127.1, 88.8)
- moved C14 42.6 mm to (126.5, 80.3)
- moved C15 42.6 mm to (123.4, 83.0)
- moved U2 42.6 mm to (127.5, 84.5)
- moved C13 42.6 mm to (124.9, 83.0)
- moved C16 42.6 mm to (124.9, 86.1)
- moved R12 42.6 mm to (131.6, 82.8)
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Connections:
- J1 pad 1: GND -> +3.3V
- J1 pad 2: DOUT -> CS
- J1 pad 3: SCLK -> DIN
- J1 pad 4: DIN -> DOUT
- J1 pad 6: CS -> SCLK
- J1 pad 7: +3.3V -> GND
- J3 pad 1: SENSE- -> IN-SENSE-
- J3 pad 2: SENSE+ -> IN-SENSE+
Routing:
- net +3.3V: track 42.4 -> 24.2 mm, vias 3 -> 2
- net SCLK: track 0.00 -> 7.39 mm
- net GND: track 46.4 -> 40.5 mm, vias 12 -> 16
- net SYNC: track 0.00 -> 5.81 mm
- net DIN: track 0.00 -> 5.40 mm
- net DOUT: track 0.00 -> 5.11 mm
- net IN-OUT-: track 8.65 -> 13.7 mm
- net IN-OUT+: track 8.86 -> 13.9 mm
- net IN-SENSE-: track 0.00 -> 4.79 mm
- net IN-SENSE+: track 0.00 -> 4.79 mm
- net +6V: track 9.50 -> 5.60 mm, vias 2 -> 0
- net Net-(U1-~{CS}): track 16.4 -> 18.2 mm
- net Net-(IC2-COMP): track 3.93 -> 2.66 mm
- net Net-(IC2-SS): track 1.63 -> 2.47 mm, vias 2 -> 0
- net Net-(U1-P2): track 33.1 -> 33.9 mm
Other:
- board text added: "+3.3V"
- board text added: "+5VA"
- board text added: "SIGNAL"

Commit message: [PCB V2]
Parts:
- removed FID1, FID2, FID3, FID4, FID5, FID6: Fiducial, Fiducial:Fiducial_1.5mm_Mask3mm
- added G***: LOGO, LOGO, F.Cu at (170.4, 89.0)
- added G***: LOGO, LOGO, F.Cu at (164.4, 109.4)
- added G***: LOGO, LOGO, B.Cu at (168.6, 78.7)
- added TP11: TestPoint, TestPoint:TestPoint_Pad_D1.5mm, F.Cu at (123.5, 89.0)
- added TP12: TestPoint, TestPoint:TestPoint_Pad_D1.5mm, F.Cu at (128.1, 77.9)
- added TP13: TestPoint, TestPoint:TestPoint_Pad_D1.5mm, F.Cu at (133.6, 81.9)
- added TP14: TestPoint, TestPoint:TestPoint_Pad_D1.5mm, B.Cu at (129.5, 91.5)
- added TP15: TestPoint, TestPoint:TestPoint_Pad_D1.5mm, B.Cu at (130.9, 97.9)
- added TP16: TestPoint, TestPoint:TestPoint_Pad_D1.5mm, B.Cu at (133.0, 94.4)
- added TP17: TestPoint, TestPoint:TestPoint_Pad_D1.5mm, F.Cu at (129.9, 88.6)
- added TP18: TestPoint, TestPoint:TestPoint_Pad_D1.5mm, B.Cu at (155.5, 91.0)
- added TP2: TestPoint, TestPoint:TestPoint_Pad_D1.5mm, B.Cu at (151.6, 95.7)
- added TP4: TestPoint, TestPoint:TestPoint_Pad_D1.5mm, F.Cu at (138.3, 105.0)
- added TP5: TestPoint, TestPoint:TestPoint_Pad_D1.5mm, F.Cu at (122.9, 78.0)
Connections:
- net Net-(IC2-COMP) renamed /Project Architecture/TPS61086_3.3V_to_6V/COMP
- net Net-(IC2-SS) renamed /Project Architecture/TPS61086_3.3V_to_6V/SS
- net Net-(U2-PG) renamed /Project Architecture/LT3042_6V_5VA/PG
Routing:
- net GND: track 40.5 -> 37.6 mm
- net /Project Architecture/LT3042_6V_5VA/SET: track 4.11 -> 6.58 mm
- net /Project Architecture/TPS61086_3.3V_to_6V/COMP: track 2.66 -> 4.78 mm, vias 0 -> 1
- net /Project Architecture/TPS61086_3.3V_to_6V/FB: track 3.57 -> 5.66 mm, vias 0 -> 1
- net /Project Architecture/LT3042_6V_5VA/PGFB: track 2.77 -> 4.80 mm
- net /Project Architecture/LT3042_6V_5VA/PG: track 2.03 -> 4.05 mm
- net +5VA: track 13.1 -> 14.8 mm
- net MCLK1: track 7.07 -> 8.44 mm, vias 0 -> 1
- net P3: track 4.04 -> 5.39 mm, vias 0 -> 1
- net /Project Architecture/TPS61086_3.3V_to_6V/SS: track 2.47 -> 3.81 mm, vias 0 -> 1
Other:
- board text added: "3.3V"
- board text added: "6V"
- board text added: "AD7190"
- board text added: "BLACk"
- board text added: "COMP"
- board text added: "CS"
- board text added: "DIN"
- board text added: "DOUT"
- board text added: "FB"
- board text added: "GND"
- board text added: "GREEN"
- board text added: "MCLK1"
- board text added: "OPEN_WEIGHT"
- board text added: "P3"
- board text added: "PG"
- board text added: "PGFB"
- board text added: "RED"
- board text added: "SCLK"
- board text added: "SET"
- board text added: "SS"
- board text added: "SYNC"
- board text added: "TPS6108"
- board text added: "WHITH"

Commit message: [PCB V3]
Routing:
- net +3.3V: track 24.2 -> 23.4 mm
- net GND: track 37.6 -> 38.2 mm, vias 16 -> 54
- net Net-(U1-P2): track 33.9 -> 33.3 mm

Commit message: [PCB V4]
Changed lines of the file:
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@@
-	)
-	(arc
-		(start 144.005 87.295)
-		(mid 144.002928 87.3)
-		(end 144.005 87.305)
-		(width 0.2)
-		(layer "F.Cu")
-		(net 3)
 	)
 	(arc
