File: Cellule_de_force_V2.kicad_pcb (KiCad board)
At the start: 4 copper layers, 57 x 50.8 mm, 73 parts, among them IC2 TPS61086DRCR, J1 Conn_01x07_Pin, J3 691408720004B, Q1 SI2303CDS-T1-GE3, U1 AD7190WBRUZ, U2 LT3042IMSE, Y2 CSTCR4M91G53-R0

Commit message: Save KiCad 10 design work (schematic + PCB) since March
Co-Authored-By: Claude Opus 5.5 <noreply@anthropic.com>
Parts:
- removed the G*** at (170.4, 89.0)
- removed the G*** at (164.4, 109.4)
- removed the G*** at (168.6, 78.7)
- removed J3: 691408720004B, 691408720004B:691408720004B
- added C27: 0.01µF, Capacitor_SMD:C_0603_1608Metric, F.Cu at (151.1, 84.6)
- added C28: 0.1µF, Capacitor_SMD:C_0603_1608Metric, F.Cu at (152.7, 86.2)
- added C29: 0.01µF, Capacitor_SMD:C_0603_1608Metric, F.Cu at (154.3, 84.7)
- added G***: LOGO, LOGO, F.Cu at (166.9, 98.4)
- added G***: LOGO, LOGO, B.Cu at (163.7, 102.6)
- added J2: 21033213501, 21033213501:21033213501, F.Cu at (135.7, 76.9)
- added J4: 21033213501, 21033213501:21033213501, F.Cu at (156.8, 76.9)
- added R4: 100Ω, Resistor_SMD:R_0603_1608Metric, F.Cu at (151.8, 82.4)
- added R5: 100Ω, Resistor_SMD:R_0603_1608Metric, F.Cu at (153.5, 82.4)
- C18: value 100nF -> 0.1uF
- TP11, TP12, TP13, TP17, TP4, TP5: moved to B.Cu
- moved R11 32.5 mm to (163.7, 103.1), turned to 180 degrees
- moved R16 30.7 mm to (163.7, 104.6), turned to 0 degrees
- moved D2 30.5 mm to (160.7, 103.1), turned to 0 degrees
- moved R3 29.0 mm to (163.7, 106.1), turned to 0 degrees
- moved D4 28.6 mm to (160.7, 104.6), turned to 0 degrees
- moved D1 26.7 mm to (160.7, 106.1), turned to 0 degrees
- moved TP12 6.04 mm to (131.2, 83.1), turned to 180 degrees
- moved C9 5.54 mm to (149.5, 83.2)
- moved C5 5.43 mm to (148.0, 84.7)
- moved C7 5.35 mm to (146.5, 83.2)
- moved TP5 4.90 mm to (127.1, 80.5), turned to 180 degrees
- moved C12 4.85 mm to (156.3, 94.5)
- moved TP4 4.79 mm to (142.9, 104.0), turned to 180 degrees
- moved TP11 4.48 mm to (127.1, 91.7), turned to 180 degrees
- moved TP14 4.14 mm to (133.6, 92.3)
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Connections:
- C10 pad 2: OUT+ -> OUT+2
- C6 pad 1: OUT+ -> OUT+2
- C6 pad 2: OUT- -> OUT-2
- C8 pad 1: OUT- -> OUT-2
- R1 pad 1: IN-OUT+ -> /Project Architecture/AD7910_Weight_sensor/IN-OUT+2
- R1 pad 2: OUT+ -> OUT+2
- R2 pad 1: IN-OUT- -> /Project Architecture/AD7910_Weight_sensor/IN-OUT-2
- R2 pad 2: OUT- -> OUT-2
- U1 pad 11: unconnected-(U1-AIN1-Pad11) -> OUT-
- U1 pad 12: unconnected-(U1-AIN2-Pad12) -> OUT+
- U1 pad 13: OUT+ -> OUT+2
- U1 pad 14: OUT- -> OUT-2
- U1 pad 17: OUT- -> SENSE-
Routing:
- net SENSE+: track 19.9 -> 56.7 mm, vias 16 -> 12
- net +3.3V: track 23.4 -> 49.6 mm, vias 2 -> 4
- net SENSE-: track 22.6 -> 41.4 mm
- net GND: track 37.1 -> 48.6 mm, vias 54 -> 97
- net /Project Architecture/Connecteur/IN-OUT+2: track 0.00 -> 10.1 mm
- net /Project Architecture/Connecteur/IN-OUT-2: track 0.00 -> 7.51 mm
- net OUT-2: track 0.00 -> 7.51 mm
- net /Project Architecture/LT3042_6V_5VA/SET: track 6.71 -> 0.00 mm, vias 0 -> 1
- net IN-OUT+: track 13.7 -> 7.50 mm
- net OUT+2: track 0.00 -> 5.61 mm
- net +6V: track 5.53 -> 0.00 mm, vias 0 -> 1
- net IN-SENSE-: track 4.76 -> 0.00 mm
- net IN-SENSE+: track 4.76 -> 0.00 mm
- net IN-OUT-: track 13.5 -> 9.56 mm
- net Net-(U1-P2): track 33.3 -> 29.7 mm
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- added copper zone on F.Cu, net /Project Architecture/LT3042_6V_5VA/SET
- removed copper zone on In2.Cu, net SENSE+
Other:
- board size 57 x 50.8 mm -> 54 x 48 mm
- board text added: "5VA"
- board text added: "BLACK"
- board text added: "INPUT-1"
- board text added: "INPUT-2"
- board text added: "WHITE"
- board text removed: "BLACk"
- board text removed: "OPEN_WEIGHT"
- board text removed: "WHITH"
