File: Section C - TItle C.kicad_sch (KiCad schematic)
At the start: 16 parts, among them U2 LT3042IMSE

Commit message: [PCB V3]
Changed lines of the file:
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@@
 		)
 	)
-	(text_box "IN (pins 1-2) : entrée d'alimentation du LT3042 (6V), à découpler avec CIN.\n\nEN/UV (pin 3) : active/désactive le régulateur et permet un seuil UVLO (souvent relié à IN pour \"toujours ON\").\n\nPG (pin 4) : sortie Power-Good open-collector (nécessite une résistance pull-up).\n\nILIM (pin 5) : programmation/monitoring de la limite de courant (souvent à GND si non utilisé).\n\nPGFB (pin 6) : entrée qui fixe le seuil de Power-Good via un pont diviseur depuis VOUT.\n\nSET (pin 7) : règle la tension de sortie via RSET (et CSET réduit le bruit/soft-start).\n\nGND (pin 8) : masse de référence du circuit.\n\nOUTS (pin 9) : sense Kelvin de la sortie (à relier au + de COUT / point de charge).\n\nOUT (pin 10) : sortie régulée (5V), à découpler avec COUT.\n\nEPAD (pad exposé) : masse + dissipation thermique (à souder sur plan GND)."
+	(text_box "IN (pins 1-2): LT3042 power input (6V), to be decoupled with CIN.\n\nEN/UV (pin 3): enables/disables the regulator and allows an UVLO threshold (often tied to IN for \"always ON\").\n\nPG (pin 4): open-collector Power-Good output (requires a pull-up resistor).\n\nILIM (pin 5): current limit programming/monitoring (often tied to GND if unused).\n\nPGFB (pin 6): input that sets the Power-Good threshold via a resistor divider from VOUT.\n\nSET (pin 7): sets the output voltage via RSET (and CSET reduces noise / provides soft-start).\n\nGND (pin 8): circuit ground reference.\n\nOUTS (pin 9): Kelvin output sense (to be connected to the + of COUT / load point).\n\nOUT (pin 10): regulated output (5V), to be decoupled with COUT.\n\nEPAD (exposed pad): ground + thermal dissipation (to be soldered to the GND plane)."
 		(exclude_from_sim no)
 		(at 52.07 91.44 0)
@@
 	(wire
 		(pts
+			(xy 337.82 129.54) (xy 340.36 129.54)
+		)
+		(stroke
+			(width 0)
+			(type default)
+		)
+	)
+	(wire
+		(pts
 			(xy 261.62 115.57) (xy 267.97 115.57)
 		)
@@
 		(pts
 			(xy 214.63 123.19) (xy 203.2 123.19)
+		)
+		(stroke
+			(width 0)
+			(type default)
+		)
+	)
+	(wire
+		(pts
+			(xy 337.82 123.19) (xy 340.36 123.19)
 		)
 		(stroke
@@
 	(symbol
 		(lib_id "Connector:TestPoint")
-		(at 339.09 127 270)
+		(at 340.36 129.54 270)
 		(unit 1)
 		(exclude_from_sim no)
@@
 		(fields_autoplaced yes)
 		(property "Reference" "TP11"
-			(at 344.17 125.7299 90)
+			(at 345.44 128.2699 90)
 			(effects
 				(font
@@
 		)
 		(property "Value" "TestPoint"
-			(at 344.17 128.2699 90)
+			(at 345.44 130.8099 90)
 			(effects
 				(font
@@
 		)
 		(property "Footprint" "TestPoint:TestPoint_Pad_D1.5mm"
-			(at 339.09 132.08 0)
+			(at 340.36 134.62 0)
 			(effects
 				(font
@@
 		)
 		(property "Datasheet" "~"
-			(at 339.09 132.08 0)
+			(at 340.36 134.62 0)
 			(effects
 				(font
@@
 		)
 		(property "Description" "test point"
-			(at 339.09 127 0)
+			(at 340.36 129.54 0)
 			(effects
 				(font
@@
 	(symbol
 		(lib_id "Connector:TestPoint")
-		(at 339.09 120.65 270)
+		(at 340.36 123.19 270)
 		(unit 1)
 		(exclude_from_sim no)
@@
 		(fields_autoplaced yes)
 		(property "Reference" "TP10"
-			(at 344.17 119.3799 90)
+			(at 345.44 121.9199 90)
 			(effects
 				(font
@@
 		)
 		(property "Value" "TestPoint"
-			(at 344.17 121.9199 90)
+			(at 345.44 124.4599 90)
 			(effects
 				(font
@@
 		)
 		(property "Footprint" "TestPoint:TestPoint_Pad_D1.5mm"
-			(at 339.09 125.73 0)
+			(at 340.36 128.27 0)
 			(effects
 				(font
@@
 		)
 		(property "Datasheet" "~"
-			(at 339.09 125.73 0)
+			(at 340.36 128.27 0)
 			(effects
 				(font
@@
 		)
 		(property "Description" "test point"
-			(at 339.09 120.65 0)
+			(at 340.36 123.19 0)
 			(effects
 				(font
@@
 	(symbol
 		(lib_id "power:+6V")
-		(at 339.09 127 90)
+		(at 337.82 129.54 90)
 		(unit 1)
 		(exclude_from_sim no)
@@
 		(dnp no)
 		(property "Reference" "#PWR021"
-			(at 342.9 127 0)
+			(at 341.63 129.54 0)
 			(effects
 				(font
@@
 		)
 		(property "Value" "+6V"
-			(at 337.312 125.476 90)
+			(at 336.042 128.016 90)
 			(effects
 				(font
@@
 		)
 		(property "Footprint" ""
-			(at 339.09 127 0)
+			(at 337.82 129.54 0)
 			(effects
 				(font
@@
 		)
 		(property "Datasheet" ""
-			(at 339.09 127 0)
+			(at 337.82 129.54 0)
 			(effects
 				(font
@@
 		)
 		(property "Description" "Power symbol creates a global label with name \"+6V\""
-			(at 339.09 127 0)
+			(at 337.82 129.54 0)
 			(effects
 				(font
@@
 	(symbol
 		(lib_id "power:+5VA")
-		(at 339.09 120.65 90)
+		(at 337.82 123.19 90)
 		(unit 1)
 		(exclude_from_sim no)
@@
 		(dnp no)
 		(property "Reference" "#PWR017"
-			(at 342.9 120.65 0)
+			(at 341.63 123.19 0)
 			(effects
 				(font
@@
 		)
 		(property "Value" "+5VA"
-			(at 339.09 119.126 90)
+			(at 337.82 121.666 90)
 			(effects
 				(font
@@
 		)
 		(property "Footprint" ""
-			(at 339.09 120.65 0)
+			(at 337.82 123.19 0)
 			(effects
 				(font
@@
 		)
 		(property "Datasheet" ""
-			(at 339.09 120.65 0)
+			(at 337.82 123.19 0)
 			(effects
 				(font
@@
 		)
 		(property "Description" "Power symbol creates a global label with name \"+5VA\""
-			(at 339.09 120.65 0)
-			(effects
-				(font
+			(at 337.82 123.19 0)
+			(effects
+				(font
