File: Section C - TItle C.kicad_sch (KiCad schematic)
At the start: 16 parts, among them U2 LT3042IMSE

Commit message: [PCB V4]
Other:
- note added: "Analog Devices"
- note added: "LT3042"
- note removed: "Flexible I/O source configuration"
- note removed: "Flexible I/O worked examples"
- note removed: "References:"
- moved on the sheet: C14, C16, D4, R14, R16, R9, U2
