File: Power - Sequencing.kicad_sch (KiCad schematic)
At the start: 0 parts

Commit message: [PCB V4]
Changed lines of the file:
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@@
 		)
 	)
-	(text_box "??"
+	(text_box "LT3042"
 		(exclude_from_sim no)
 		(at 31.75 54.483 0)
@@
 		(stroke
 			(width 0)
-			(type default)
+			(type solid)
 			(color 0 0 0 1)
 		)
@@
 		)
 	)
-	(text_box "+V??"
+	(text_box "+5VA"
 		(exclude_from_sim no)
 		(at 15.24 54.483 0)
@@
 		(stroke
 			(width 0)
-			(type default)
+			(type solid)
 			(color 0 0 0 1)
 		)
