File: Section B - TItle B.kicad_sch (KiCad schematic)
At the start: 3 parts, among them IC2 TPS61086DRCR

Commit message: [Finish schématique]
Parts:
- added C17: 2.2nF, Capacitor_SMD:C_0603_1608Metric, symbol Device:C
- added C18: 100nF, Capacitor_SMD:C_0603_1608Metric, symbol Device:C
- added C19, C20, C21: 10µF, Capacitor_SMD:C_0603_1608Metric, symbol Device:C
- added C22: 1µF, Capacitor_SMD:C_0603_1608Metric, symbol Device:C
- added D3: PMEG2010AEH, Diode_SMD:D_SOD-123F, symbol Diode:PMEG2010AEH
- added L1: 7447785004, 7447785004, symbol 7447785004:7447785004
- added R18: 37.4kΩ, Resistor_SMD:R_0603_1608Metric, symbol Device:R
- added TP19, TP20, TP21: TestPoint, TestPoint:TestPoint_Pad_D2.0mm, symbol Connector:TestPoint
Connections:
- net +3.3V_IN: now also IC2.3 (EN), C21.1, C22.1, L1.1, TP21.1
- net +6V_OUT: now also C19.1, C20.1, D3.1 (K), TP20.1; no longer IC2.6 (SW_1), IC2.7 (SW_2)
- net GND: now also C17.2, C18.2, C19.2, C20.2, C21.2, C22.2
- net at IC2.1 (COMP): now also R18.2
- net at IC2.10 (SS): now also C18.1
- net FB: now reaches IC2.2 (FB), R15.2, R17.1
- net FB: now also TP19.1
- new net: C17.1, R18.1
- new net: D3.2 (A), IC2.6 (SW_1), IC2.7 (SW_2), L1.2
Other:
- moved on the sheet: R15, R17

Commit message: [Finish schématiq]
Parts:
- added TP22: TestPoint, TestPoint:TestPoint_Pad_D2.0mm, symbol Connector:TestPoint
Connections:
- net GND: now also TP22.1
Other:
- moved on the sheet: C17, C18, C19, C20, C21, C22, D3, IC2, L1, R15, R17, R18

Commit message: [PCB fini]
Parts:
- L1: footprint 7447785004 -> 7447785004:7447785004

Commit message: [PCB 4 layer]
Parts:
- added D1: LED, LED_SMD:LED_0603_1608Metric, symbol Device:LED
- added R3: 100Ω, Resistor_SMD:R_0603_1608Metric, symbol Device:R
- IC2: footprint TPS16412DRCR -> TPS61086DRCR:TPS16412DRCR
Connections:
- net +3.3V_IN: no longer C21.1, C22.1, IC2.3 (EN), IC2.8 (IN), L1.1
- net +6V_OUT: no longer C19.1, C20.1, D3.1 (K), R17.2
- net GND: now also D1.1 (K)
- new net: D1.2 (A), R3.1
- new net +3.3V: C21.1, C22.1, IC2.3 (EN), IC2.8 (IN), L1.1, R3.2
- new net +6V: C19.1, C20.1, D3.1 (K), R17.2
Changed lines of the file:
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@@
+	)
+	(junction
+		(at 172.72 113.03)
+		(diameter 0)
+		(color 0 0 0 0)
 	)
 	(junction
@@
 	)
 	(junction
+		(at 187.96 143.51)
+		(diameter 0)
+		(color 0 0 0 0)
+	)
+	(junction
 		(at 207.01 128.27)
 		(diameter 0)
@@
 	(wire
 		(pts
+			(xy 172.72 128.27) (xy 172.72 143.51)
+		)
+		(stroke
+			(width 0)
+			(type default)
+		)
+	)
+	(wire
+		(pts
 			(xy 250.19 113.03) (xy 255.27 113.03)
 		)
@@
 	(wire
 		(pts
+			(xy 172.72 113.03) (xy 187.96 113.03)
+		)
+		(stroke
+			(width 0)
+			(type default)
+		)
+	)
+	(wire
+		(pts
 			(xy 247.65 143.51) (xy 255.27 143.51)
 		)
@@
 	(wire
 		(pts
+			(xy 172.72 143.51) (xy 187.96 143.51)
+		)
+		(stroke
+			(width 0)
+			(type default)
+		)
+	)
+	(wire
+		(pts
 			(xy 207.01 119.38) (xy 193.04 119.38)
 		)
@@
 	(wire
 		(pts
-			(xy 182.88 113.03) (xy 187.96 113.03)
+			(xy 168.91 113.03) (xy 172.72 113.03)
 		)
 		(stroke
@@
 			)
 		)
-		(property "Value" "+6V_OUT"
-			(at 279.4 109.728 0)
+		(property "Value" "+6V"
+			(at 288.29 108.712 0)
 			(effects
 				(font
@@
 			)
 		)
-		(property "Footprint" "TPS16412DRCR"
+		(property "Footprint" "TPS61086DRCR:TPS16412DRCR"
 			(at 233.68 201.6 0)
 			(effects
@@
 				)
 				(justify left)
+				(hide yes)
 			)
 		)
@@
 		)
 		(property "Value" "37.4kΩ"
-			(at 249.682 132.08 90)
-			(effects
-				(font
-					(size 1.27 1.27)
+			(at 247.65 132.08 90)
+			(effects
+				(font
+					(size 1.016 1.016)
 				)
 			)
@@
 	)
 	(symbol
+		(lib_id "Device:R")
+		(at 172.72 116.84 180)
+		(unit 1)
+		(exclude_from_sim no)
+		(in_bom yes)
+		(on_board yes)
+		(dnp no)
+		(property "Reference" "R3"
+			(at 170.688 117.856 90)
+			(effects
+				(font
+					(size 1.27 1.27)
+				)
+			)
+		)
+		(property "Value" "100Ω"
+			(at 172.72 116.84 90)
+			(effects
+				(font
+					(size 1.016 1.016)
+				)
+			)
+		)
+		(property "Footprint" "Resistor_SMD:R_0603_1608Metric"
+			(at 174.498 116.84 90)
+			(effects
+				(font
+					(size 1.27 1.27)
+				)
+				(hide yes)
+			)
+		)
+		(property "Datasheet" "~"
+			(at 172.72 116.84 0)
+			(effects
+				(font
+					(size 1.27 1.27)
+				)
+				(hide yes)
+			)
+		)
+		(property "Description" "Resistor"
+			(at 172.72 116.84 0)
+			(effects
+				(font
+					(size 1.27 1.27)
+				)
+				(hide yes)
+			)
+		)
+		(pin "2"
+		)
+		(pin "1"
+		)
+		(instances
+			(project "Cellule_de_force_V2"
+				(path "/f9e05184-c88b-4a88-ae9c-ab2bdb32be7c/c5103ceb-5325-4a84-a025-9638a412984e/d6110ee2-516c-48c1-b80a-d0f1701ed49f"
+					(reference "R3")
+					(unit 1)
+				)
+			)
+		)
+	)
+	(symbol
 		(lib_id "power:+3.3V")
-		(at 182.88 113.03 0)
+		(at 168.91 113.03 0)
 		(unit 1)
 		(exclude_from_sim no)
@@
 		(dnp no)
 		(property "Reference" "#PWR026"
-			(at 182.88 116.84 0)
-			(effects
-				(font
-					(size 1.27 1.27)
-				)
-				(hide yes)
-			)
-		)
-		(property "Value" "+3.3V_IN"
-			(at 179.07 108.966 0)
+			(at 168.91 116.84 0)
+			(effects
+				(font
+					(size 1.27 1.27)
+				)
+				(hide yes)
+			)
+		)
+		(property "Value" "+3.3V"
+			(at 165.1 108.966 0)
 			(effects
 				(font
@@
 		)
 		(property "Footprint" ""
-			(at 182.88 113.03 0)
+			(at 168.91 113.03 0)
 			(effects
 				(font
@@
 		)
 		(property "Datasheet" ""
-			(at 182.88 113.03 0)
+			(at 168.91 113.03 0)
 			(effects
 				(font
@@
 		)
 		(property "Description" "Power symbol creates a global label with name \"+3.3V\""
-			(at 182.88 113.03 0)
+			(at 168.91 113.03 0)
 			(effects
 				(font
@@
 				(path "/f9e05184-c88b-4a88-ae9c-ab2bdb32be7c/c5103ceb-5325-4a84-a025-9638a412984e/d6110ee2-516c-48c1-b80a-d0f1701ed49f"
 					(reference "#PWR026")
+					(unit 1)
+				)
+			)
+		)
+	)
+	(symbol
+		(lib_id "Device:LED")
+		(at 172.72 124.46 90)
+		(unit 1)
+		(exclude_from_sim no)
+		(in_bom yes)
+		(on_board yes)
+		(dnp no)
+		(property "Reference" "D1"
+			(at 170.688 124.206 0)
+			(effects
+				(font
+					(size 1.27 1.27)
+				)
+			)
+		)
+		(property "Value" "LED"
+			(at 170.942 127.508 0)
+			(effects
+				(font
+					(size 1.27 1.27)
+				)
+			)
+		)
+		(property "Footprint" "LED_SMD:LED_0603_1608Metric"
+			(at 172.72 124.46 0)
+			(effects
+				(font
+					(size 1.27 1.27)
+				)
+				(hide yes)
+			)
+		)
+		(property "Datasheet" "~"
+			(at 172.72 124.46 0)
+			(effects
+				(font
+					(size 1.27 1.27)
+				)
+				(hide yes)
+			)
+		)
+		(property "Description" "Light emitting diode"
+			(at 172.72 124.46 0)
+			(effects
+				(font
+					(size 1.27 1.27)
+				)
+				(hide yes)
+			)
+		)
+		(property "Sim.Pins" "1=K 2=A"
+			(at 172.72 124.46 0)
+			(effects
+				(font
+					(size 1.27 1.27)
+				)
+				(hide yes)
+			)
+		)
+		(pin "2"
+		)
+		(pin "1"
+		)
+		(instances
+			(project "Cellule_de_force_V2"
+				(path "/f9e05184-c88b-4a88-ae9c-ab2bdb32be7c/c5103ceb-5325-4a84-a025-9638a412984e/d6110ee2-516c-48c1-b80a-d0f1701ed49f"
+					(reference "D1")
 					(unit 1)
 				)
@@
 		)
 		(property "Value" "18kΩ"
-			(at 257.302 124.206 90)
-			(effects
-				(font
-					(size 1.27 1.27)
+			(at 255.27 124.206 90)
+			(effects
+				(font
+					(size 1.016 1.016)
 				)
 			)
@@
 				)
 				(justify left)
+				(hide yes)
 			)
 		)
@@
 		)
 		(property "Value" "69.8kΩ"
-			(at 257.302 116.84 90)
-			(effects
-				(font
-					(size 1.27 1.27)
-				)
-			)
+			(at 255.27 116.84 90)
+			(effects
+				(font
+					(size 1.016 1.016)
+				)
+			)

Commit message: [PCB V1]
Parts:
- removed TP19, TP20, TP21, TP22: TestPoint, TestPoint:TestPoint_Pad_D2.0mm, symbol Connector:TestPoint
- added TP14, TP15, TP16: TestPoint, TestPoint:TestPoint_Pad_D1.5mm, symbol Connector:TestPoint
Connections:
- net FB: now also TP14.1
- net COMP: now reaches IC2.1 (COMP), R18.2
- net COMP: now also TP16.1
- net SS: now reaches C18.1, IC2.10 (SS)
- net SS: now also TP15.1

Commit message: [PCB V3]
Other:
- moved on the sheet: C21, C22, D1, R3

Commit message: [PCB V4]
Parts:
- C18: value 100nF -> 0.1uF
