File: Section D - TItle D.kicad_sch (KiCad schematic)
At the start: 0 parts

Commit message: [Finish schématique]
Parts:
- added J1, J2, J3, J4: Conn_01x02_Pin, Connector_PinHeader_2.54mm:PinHeader_1x02_P2.54mm_Vertical, symbol Connector:Conn_01x02_Pin
- added J5: Conn_01x04_Socket, Connector_PinSocket_2.54mm:PinSocket_1x04_P2.54mm_Vertical, symbol Connector:Conn_01x04_Socket
- added J6: Conn_01x05_Pin, Connector_PinSocket_2.54mm:PinSocket_1x05_P2.54mm_Vertical, symbol Connector:Conn_01x05_Pin
Connections:
- new net +3.3V_IN: J1.1 (Pin_1), J3.1 (Pin_1), J3.2 (Pin_2)
- new net +5VA_IN: J4.1 (Pin_1)
- new net +5VA_OUT: J4.2 (Pin_2)
- new net +6V_IN: J2.2 (Pin_2)
- new net +6V_OUT: J2.1 (Pin_1)
- new net CS: J6.1 (Pin_1)
- new net DIN: J6.4 (Pin_4)
- new net DOUT: J6.5 (Pin_5)
- new net GND: J1.2 (Pin_2)
- new net IN-SENSE+: J5.1 (Pin_1)
- new net OUT+: J5.3 (Pin_3)
- new net OUT-: J5.4 (Pin_4)
- new net SCLK: J6.2 (Pin_2)
- new net SENSE-: J5.2 (Pin_2)
- new net SYNC: J6.3 (Pin_3)

Commit message: [Finish schématiq]
Other:
- moved on the sheet: J2, J3, J4, J5, J6

Commit message: [PCB fini]
Connections:
- net SENSE- is gone; now on net IN-SENSE+: J5.2 (Pin_2)
- net CS: now also J6.5 (Pin_5); no longer J6.1 (Pin_1)
- net DIN: now also J6.3 (Pin_3); no longer J6.4 (Pin_4)
- net DOUT: now also J6.2 (Pin_2); no longer J6.5 (Pin_5)
- net IN-SENSE+: no longer J5.1 (Pin_1)
- net SCLK: now also J6.4 (Pin_4); no longer J6.2 (Pin_2)
- net SYNC: now also J6.1 (Pin_1); no longer J6.3 (Pin_3)
- net OUT+ renamed IN-OUT-
- net OUT- renamed IN-OUT+
- new net IN-SENSE-: J5.1 (Pin_1)
Changed lines of the file:
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@@
 		)
 	)
-	(global_label "SCLK"
+	(global_label "CS"
 		(shape input)
-		(at 245.11 127 0)
+		(at 245.11 134.62 0)
 		(fields_autoplaced yes)
 		(effects
@@
 		)
 		(property "Intersheetrefs" "${INTERSHEET_REFS}"
-			(at 252.8728 127 0)
+			(at 250.5747 134.62 0)
 			(effects
 				(font
@@
 		)
 	)
-	(global_label "CS"
+	(global_label "IN-OUT-"
 		(shape input)
-		(at 245.11 124.46 0)
+		(at 274.32 129.54 180)
+		(fields_autoplaced yes)
+		(effects
+			(font
+				(size 1.27 1.27)
+			)
+			(justify right)
+		)
+		(property "Intersheetrefs" "${INTERSHEET_REFS}"
+			(at 262.6261 129.54 0)
+			(effects
+				(font
+					(size 1.27 1.27)
+				)
+				(justify right)
+				(hide yes)
+			)
+		)
+	)
+	(global_label "DIN"
+		(shape input)
+		(at 245.11 129.54 0)
 		(fields_autoplaced yes)
 		(effects
@@
 		)
 		(property "Intersheetrefs" "${INTERSHEET_REFS}"
-			(at 250.5747 124.46 0)
+			(at 251.3005 129.54 0)
 			(effects
 				(font
@@
 		)
 	)
-	(global_label "IN-SENSE+"
+	(global_label "IN-SENSE-"
 		(shape input)
 		(at 274.32 124.46 180)
@@
 		)
 	)
-	(global_label "OUT-"
+	(global_label "DOUT"
+		(shape input)
+		(at 245.11 127 0)
+		(fields_autoplaced yes)
+		(effects
+			(font
+				(size 1.27 1.27)
+			)
+			(justify left)
+		)
+		(property "Intersheetrefs" "${INTERSHEET_REFS}"
+			(at 252.9938 127 0)
+			(effects
+				(font
+					(size 1.27 1.27)
+				)
+				(justify left)
+				(hide yes)
+			)
+		)
+	)
+	(global_label "IN-OUT+"
 		(shape input)
 		(at 274.32 132.08 180)
@@
 		)
 		(property "Intersheetrefs" "${INTERSHEET_REFS}"
-			(at 266.1338 132.08 0)
+			(at 262.6261 132.08 0)
 			(effects
 				(font
@@
 		)
 	)
-	(global_label "SENSE-"
+	(global_label "SCLK"
+		(shape input)
+		(at 245.11 132.08 0)
+		(fields_autoplaced yes)
+		(effects
+			(font
+				(size 1.27 1.27)
+			)
+			(justify left)
+		)
+		(property "Intersheetrefs" "${INTERSHEET_REFS}"
+			(at 252.8728 132.08 0)
+			(effects
+				(font
+					(size 1.27 1.27)
+				)
+				(justify left)
+				(hide yes)
+			)
+		)
+	)
+	(global_label "IN-SENSE+"
 		(shape input)
 		(at 274.32 127 180)
@@
 		)
 		(property "Intersheetrefs" "${INTERSHEET_REFS}"
-			(at 263.7149 127 0)
-			(effects
-				(font
-					(size 1.27 1.27)
-				)
-				(justify right)
-				(hide yes)
-			)
-		)
-	)
-	(global_label "OUT+"
-		(shape input)
-		(at 274.32 129.54 180)
-		(fields_autoplaced yes)
-		(effects
-			(font
-				(size 1.27 1.27)
-			)
-			(justify right)
-		)
-		(property "Intersheetrefs" "${INTERSHEET_REFS}"
-			(at 266.1338 129.54 0)
+			(at 260.2072 127 0)
 			(effects
 				(font
@@
 	(global_label "SYNC"
 		(shape input)
-		(at 245.11 129.54 0)
+		(at 245.11 124.46 0)
 		(fields_autoplaced yes)
 		(effects
@@
 		)
 		(property "Intersheetrefs" "${INTERSHEET_REFS}"
-			(at 252.9938 129.54 0)
+			(at 252.9938 124.46 0)
 			(effects
 				(font
-					(size 1.27 1.27)
-				)
-				(justify left)
-				(hide yes)
-			)
-		)
-	)
-	(global_label "DIN"
-		(shape input)
-		(at 245.11 132.08 0)
-		(fields_autoplaced yes)
-		(effects
-			(font
-				(size 1.27 1.27)
-			)
-			(justify left)
-		)
-		(property "Intersheetrefs" "${INTERSHEET_REFS}"
-			(at 251.3005 132.08 0)
-			(effects
-				(font
-					(size 1.27 1.27)
-				)
-				(justify left)
-				(hide yes)
-			)
-		)
-	)
-	(global_label "DOUT"
-		(shape input)
-		(at 245.11 134.62 0)
-		(fields_autoplaced yes)
-		(effects
-			(font
-				(size 1.27 1.27)
-			)
-			(justify left)
-		)
-		(property "Intersheetrefs" "${INTERSHEET_REFS}"
-			(at 252.9938 134.62 0)
-			(effects
-				(font

Commit message: [PCB 4 layer]
Parts:
- removed J1, J2, J3, J4: Conn_01x02_Pin, Connector_PinHeader_2.54mm:PinHeader_1x02_P2.54mm_Vertical, symbol Connector:Conn_01x02_Pin
- removed J5: Conn_01x04_Socket, Connector_PinSocket_2.54mm:PinSocket_1x04_P2.54mm_Vertical, symbol Connector:Conn_01x04_Socket
- removed J6: Conn_01x05_Pin, Connector_PinSocket_2.54mm:PinSocket_1x05_P2.54mm_Vertical, symbol Connector:Conn_01x05_Pin
- added H5: WE-SHC_THT-FRAME, WE-SHC_THT-FRAME:WE-SHC_THT-FRAME_36503205, symbol WE-SHC_THT-FRAME:WE-SHC_THT-FRAME
- added J1: Conn_01x07_Pin, Connector_JST:JST_XH_B7B-XH-AM_1x07_P2.50mm_Vertical, symbol Connector:Conn_01x07_Pin
- added J3: 691408720004B, 691408720004B:691408720004B, symbol 691408720004B:691408720004B
Connections:
- net CS: now also J1.6 (Pin_6)
- net DIN: now also J1.4 (Pin_4)
- net DOUT: now also J1.2 (Pin_2)
- net GND: now also H5.1, H5.10, H5.11, H5.12, H5.13, H5.14, H5.15, H5.16, H5.17, H5.2, H5.3, H5.4, H5.5, H5.6, H5.7, H5.9, J1.1 (Pin_1)
- net IN-OUT+: now also J3.3, J3.A3
- net IN-OUT-: now also J3.4, J3.A4
- net IN-SENSE+: now also J3.2, J3.A2
- net IN-SENSE-: now also J3.1, J3.A1
- net SCLK: now also J1.3 (Pin_3)
- net SYNC: now also J1.5 (Pin_5)
- new net +3.3V: J1.7 (Pin_7)

Commit message: [PCB V1]
Connections:
- net +3.3V: now also J1.1 (Pin_1); no longer J1.7 (Pin_7)
- net CS: now also J1.2 (Pin_2); no longer J1.6 (Pin_6)
- net DIN: now also J1.3 (Pin_3); no longer J1.4 (Pin_4)
- net DOUT: now also J1.4 (Pin_4); no longer J1.2 (Pin_2)
- net GND: now also J1.7 (Pin_7); no longer J1.1 (Pin_1)
- net SCLK: now also J1.6 (Pin_6); no longer J1.3 (Pin_3)
Changed lines of the file:
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@@
+		)
+	)
+	(label "SCLK"
+		(at 190.5 114.3 0)
+		(effects
+			(font
+				(size 1.27 1.27)
+			)
+			(justify left bottom)
 		)
 	)
 	(label "CS"
-		(at 190.5 114.3 0)
+		(at 190.5 104.14 0)
 		(effects
 			(font
@@
 		)
 	)
+	(label "DOUT"
+		(at 190.5 109.22 0)
+		(effects
+			(font
+				(size 1.27 1.27)
+			)
+			(justify left bottom)
+		)
+	)
 	(label "SYNC"
 		(at 190.5 111.76 0)
@@
 		)
 	)
-	(label "DOUT"
-		(at 190.5 104.14 0)
-		(effects
-			(font
-				(size 1.27 1.27)
-			)
-			(justify left bottom)
-		)
-	)
 	(label "DIN"
-		(at 190.5 109.22 0)
+		(at 190.5 106.68 0)
 		(effects
 			(font
@@
 	(label "IN-OUT-"
 		(at 214.63 110.49 0)
-		(effects
-			(font
-				(size 1.27 1.27)
-			)
-			(justify left bottom)
-		)
-	)
-	(label "SCLK"
-		(at 190.5 106.68 0)
 		(effects
 			(font
@@
 				(justify left)
 				(hide yes)
-			)
-		)
-	)
-	(symbol
-		(lib_id "power:+3.3V")
-		(at 190.5 116.84 180)
-		(unit 1)
-		(exclude_from_sim no)
-		(in_bom yes)
-		(on_board yes)
-		(dnp no)
-		(property "Reference" "#PWR033"
-			(at 190.5 113.03 0)
-			(effects
-				(font
-					(size 1.27 1.27)
-				)
-				(hide yes)
-			)
-		)
-		(property "Value" "+3.3V"
-			(at 194.31 120.904 0)
-			(effects
-				(font
-					(size 1.27 1.27)
-				)
-				(justify left)
-			)
-		)
-		(property "Footprint" ""
-			(at 190.5 116.84 0)
-			(effects
-				(font
-					(size 1.27 1.27)
-				)
-				(hide yes)
-			)
-		)
-		(property "Datasheet" ""
-			(at 190.5 116.84 0)
-			(effects
-				(font
-					(size 1.27 1.27)
-				)
-				(hide yes)
-			)
-		)
-		(property "Description" "Power symbol creates a global label with name \"+3.3V\""
-			(at 190.5 116.84 0)
-			(effects
-				(font
-					(size 1.27 1.27)
-				)
-				(hide yes)
-			)
-		)
-		(pin "1"
-		)
-		(instances
-			(project "Cellule_de_force_V2"
-				(path "/f9e05184-c88b-4a88-ae9c-ab2bdb32be7c/c5103ceb-5325-4a84-a025-9638a412984e/ddd4b387-4aa4-48c3-b079-ffb0beb645d3"
-					(reference "#PWR033")
-					(unit 1)
-				)
 			)
 		)
@@
 	)
 	(symbol
-		(lib_id "power:GND")
-		(at 190.5 101.6 180)
+		(lib_id "power:+3.3V")
+		(at 190.5 101.6 0)
 		(unit 1)
 		(exclude_from_sim no)
@@
 		(on_board yes)
 		(dnp no)
-		(fields_autoplaced yes)
-		(property "Reference" "#PWR032"
-			(at 190.5 95.25 0)
-			(effects
-				(font
-					(size 1.27 1.27)
-				)
-				(hide yes)
-			)
-		)
-		(property "Value" "GND"
-			(at 190.5 96.52 0)
-			(effects
-				(font
-					(size 1.27 1.27)
-				)
-				(hide yes)
+		(property "Reference" "#PWR029"
+			(at 190.5 105.41 0)
+			(effects
+				(font
+					(size 1.27 1.27)
+				)
+				(hide yes)
+			)
+		)
+		(property "Value" "+3.3V"
+			(at 186.69 97.536 0)
+			(effects
+				(font
+					(size 1.27 1.27)
+				)
+				(justify left)
 			)
 		)
@@
 			)
 		)
-		(property "Description" "Power symbol creates a global label with name \"GND\" , ground"
+		(property "Description" "Power symbol creates a global label with name \"+3.3V\""
 			(at 190.5 101.6 0)
 			(effects
@@
 			(project "Cellule_de_force_V2"
 				(path "/f9e05184-c88b-4a88-ae9c-ab2bdb32be7c/c5103ceb-5325-4a84-a025-9638a412984e/ddd4b387-4aa4-48c3-b079-ffb0beb645d3"
-					(reference "#PWR032")
+					(reference "#PWR029")
 					(unit 1)
 				)
@@
 					(unit 1)
 				)
+			)
+		)
+	)
+	(symbol
+		(lib_id "power:GND")
+		(at 190.5 116.84 0)
+		(unit 1)
+		(exclude_from_sim no)
+		(in_bom yes)
+		(on_board yes)
+		(dnp no)
+		(fields_autoplaced yes)
+		(property "Reference" "#PWR030"
+			(at 190.5 123.19 0)
+			(effects
+				(font
+					(size 1.27 1.27)
+				)
+				(hide yes)
+			)
+		)
+		(property "Value" "GND"
+			(at 190.5 121.92 0)
+			(effects
+				(font
+					(size 1.27 1.27)
+				)
+				(hide yes)
+			)
+		)
+		(property "Footprint" ""
+			(at 190.5 116.84 0)
+			(effects
+				(font
+					(size 1.27 1.27)
+				)
+				(hide yes)
+			)
+		)
+		(property "Datasheet" ""
+			(at 190.5 116.84 0)
+			(effects
+				(font
+					(size 1.27 1.27)
+				)
+				(hide yes)
+			)
+		)
+		(property "Description" "Power symbol creates a global label with name \"GND\" , ground"
+			(at 190.5 116.84 0)
+			(effects
+				(font
+					(size 1.27 1.27)
+				)
+				(hide yes)
+			)
+		)
+		(pin "1"
+		)
+		(instances
+			(project "Cellule_de_force_V2"
+				(path "/f9e05184-c88b-4a88-ae9c-ab2bdb32be7c/c5103ceb-5325-4a84-a025-9638a412984e/ddd4b387-4aa4-48c3-b079-ffb0beb645d3"
+					(reference "#PWR030")
+					(unit 1)
+				)

Commit message: [PCB V3]
Other:
- moved on the sheet: H5
Changed lines of the file:
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@@
 					(size 1.27 1.27)
 				)
+				(hide yes)
 			)
 		)
@@
 	(symbol
 		(lib_id "WE-SHC_THT-FRAME:WE-SHC_THT-FRAME")
-		(at 224.79 148.59 0)
+		(at 267.97 105.41 0)
 		(unit 1)
 		(exclude_from_sim no)
@@
 		(fields_autoplaced yes)
 		(property "Reference" "H5"
-			(at 238.76 149.8599 0)
+			(at 281.94 106.6799 0)
 			(effects
 				(font
@@
 		)
 		(property "Value" "WE-SHC_THT-FRAME"
-			(at 238.76 152.3999 0)
+			(at 281.94 109.2199 0)
 			(effects
 				(font
@@
 		)
 		(property "Footprint" "WE-SHC_THT-FRAME:WE-SHC_THT-FRAME_36503205"
-			(at 224.79 148.59 0)
+			(at 267.97 105.41 0)
 			(effects
 				(font
@@
 		)
 		(property "Datasheet" ""
-			(at 224.79 148.59 0)
+			(at 267.97 105.41 0)
 			(effects
 				(font
@@
 		)
 		(property "Description" ""
-			(at 224.79 148.59 0)
+			(at 267.97 105.41 0)
 			(effects
 				(font
@@
 		)
 		(property "MF" "Wurth Electronics"
-			(at 224.79 148.59 0)
+			(at 267.97 105.41 0)
 			(effects
 				(font
@@
 		)
 		(property "Description_1" "Frame THT; 20 x 20 x 3 mm; Base material = tinplate"
-			(at 224.79 148.59 0)
+			(at 267.97 105.41 0)
 			(effects
 				(font
@@
 		)
 		(property "Package" "None"
-			(at 224.79 148.59 0)
+			(at 267.97 105.41 0)
 			(effects
 				(font
@@
 		)
 		(property "Price" "None"
-			(at 224.79 148.59 0)
+			(at 267.97 105.41 0)
 			(effects
 				(font
@@
 		)
 		(property "SnapEDA_Link" "https://www.snapeda.com/parts/36503205S/Wurth+Electronics/view-part/?ref=snap"
-			(at 224.79 148.59 0)
+			(at 267.97 105.41 0)
 			(effects
 				(font
@@
 		)
 		(property "MP" "36503205S"
-			(at 224.79 148.59 0)
+			(at 267.97 105.41 0)
 			(effects
 				(font
@@
 		)
 		(property "Purchase-URL" "https://www.snapeda.com/api/url_track_click_mouser/?unipart_id=13768814&manufacturer=Wurth Electronics&part_name=36503205S&search_term=36503205s"
-			(at 224.79 148.59 0)
+			(at 267.97 105.41 0)
 			(effects
 				(font
@@
 		)
 		(property "Availability" "In Stock"
-			(at 224.79 148.59 0)
+			(at 267.97 105.41 0)
 			(effects
 				(font
@@
 		)
 		(property "Check_prices" "https://www.snapeda.com/parts/36503205S/Wurth+Electronics/view-part/?ref=eda"
-			(at 224.79 148.59 0)
+			(at 267.97 105.41 0)
 			(effects
 				(font
@@
 	(symbol
 		(lib_id "power:GND")
-		(at 214.63 146.05 0)
+		(at 257.81 102.87 0)
 		(unit 1)
 		(exclude_from_sim no)
@@
 		(fields_autoplaced yes)
 		(property "Reference" "#PWR031"
-			(at 214.63 152.4 0)
+			(at 257.81 109.22 0)
 			(effects
 				(font
@@
 		)
 		(property "Value" "GND"
-			(at 214.63 151.13 0)
+			(at 257.81 107.95 0)
 			(effects
 				(font
@@
 		)
 		(property "Footprint" ""
-			(at 214.63 146.05 0)
+			(at 257.81 102.87 0)
 			(effects
 				(font
@@
 		)
 		(property "Datasheet" ""
-			(at 214.63 146.05 0)
+			(at 257.81 102.87 0)
 			(effects
 				(font
@@
 		)
 		(property "Description" "Power symbol creates a global label with name \"GND\" , ground"
-			(at 214.63 146.05 0)
+			(at 257.81 102.87 0)
 			(effects
 				(font
@@
 				)
 				(justify left)
-			)
-		)
+				(hide yes)
+			)
+		)
