File: Section D - TItle D.kicad_sch (KiCad schematic)
At the start: 3 parts, among them J1 Conn_01x07_Pin, J3 691408720004B

Commit message: Save KiCad 10 design work (schematic + PCB) since March
Co-Authored-By: Claude Opus 5.5 <noreply@anthropic.com>
Parts:
- removed J3: 691408720004B, 691408720004B:691408720004B, symbol 691408720004B:691408720004B
- added J2, J4: 21033213501, 21033213501, symbol 21033213501:21033213501
Connections:
- net GND: now also J2.5, J2.S1 (SHIELD), J4.5, J4.S1 (SHIELD)
- net IN-OUT+: now also J4.1
- net IN-OUT-: now also J4.2
- net IN-SENSE+: now also J2.4, J4.4
- net IN-SENSE-: now also J2.3, J4.3
- new net IN-OUT+2: J2.1
- new net IN-OUT-2: J2.2
