File: Section E - TItle E.kicad_sch (KiCad schematic)
At the start: 7 parts

Commit message: [Finish schématiq]
Parts:
- added FID4, FID5, FID6: Fiducial, Fiducial:Fiducial_1.5mm_Mask3mm, symbol Mechanical:Fiducial
Other:
- moved on the sheet: FID1, FID2, FID3, H1, H2, H3, H4

Commit message: [PCB V3]
Other:
- moved on the sheet: FID1, FID2, FID3, FID4, FID5, FID6
Changed lines of the file:
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@@
 	(symbol
 		(lib_id "Mechanical:Fiducial")
-		(at 224.79 139.7 0)
+		(at 223.52 139.7 0)
 		(unit 1)
 		(exclude_from_sim no)
@@
 		(fields_autoplaced yes)
 		(property "Reference" "FID2"
-			(at 227.33 138.4299 0)
+			(at 226.06 138.4299 0)
 			(effects
 				(font
@@
 		)
 		(property "Value" "Fiducial"
-			(at 227.33 140.9699 0)
+			(at 226.06 140.9699 0)
 			(effects
 				(font
@@
 		)
 		(property "Footprint" "Fiducial:Fiducial_1.5mm_Mask3mm"
-			(at 224.79 139.7 0)
-			(effects
-				(font
-					(size 1.27 1.27)
-				)
-				(hide yes)
-			)
-		)
-		(property "Datasheet" "~"
-			(at 224.79 139.7 0)
+			(at 223.52 139.7 0)
+			(effects
+				(font
+					(size 1.27 1.27)
+				)
+				(hide yes)
+			)
+		)
+		(property "Datasheet" "~"
+			(at 223.52 139.7 0)
 			(effects
 				(font
@@
 		)
 		(property "Description" "Fiducial Marker"
-			(at 224.79 139.7 0)
+			(at 223.52 139.7 0)
 			(effects
 				(font
@@
 	(symbol
 		(lib_id "Mechanical:Fiducial")
-		(at 224.79 144.78 0)
+		(at 223.52 144.78 0)
 		(unit 1)
 		(exclude_from_sim no)
@@
 		(fields_autoplaced yes)
 		(property "Reference" "FID3"
-			(at 227.33 143.5099 0)
+			(at 226.06 143.5099 0)
 			(effects
 				(font
@@
 		)
 		(property "Value" "Fiducial"
-			(at 227.33 146.0499 0)
+			(at 226.06 146.0499 0)
 			(effects
 				(font
@@
 		)
 		(property "Footprint" "Fiducial:Fiducial_1.5mm_Mask3mm"
-			(at 224.79 144.78 0)
-			(effects
-				(font
-					(size 1.27 1.27)
-				)
-				(hide yes)
-			)
-		)
-		(property "Datasheet" "~"
-			(at 224.79 144.78 0)
+			(at 223.52 144.78 0)
+			(effects
+				(font
+					(size 1.27 1.27)
+				)
+				(hide yes)
+			)
+		)
+		(property "Datasheet" "~"
+			(at 223.52 144.78 0)
 			(effects
 				(font
@@
 		)
 		(property "Description" "Fiducial Marker"
-			(at 224.79 144.78 0)
+			(at 223.52 144.78 0)
 			(effects
 				(font
@@
 	(symbol
 		(lib_id "Mechanical:Fiducial")
-		(at 262.89 134.62 0)
+		(at 260.35 134.62 0)
 		(unit 1)
 		(exclude_from_sim no)
@@
 		(fields_autoplaced yes)
 		(property "Reference" "FID4"
-			(at 265.43 133.3499 0)
+			(at 262.89 133.3499 0)
 			(effects
 				(font
@@
 		)
 		(property "Value" "Fiducial"
-			(at 265.43 135.8899 0)
+			(at 262.89 135.8899 0)
 			(effects
 				(font
@@
 		)
 		(property "Footprint" "Fiducial:Fiducial_1.5mm_Mask3mm"
-			(at 262.89 134.62 0)
-			(effects
-				(font
-					(size 1.27 1.27)
-				)
-				(hide yes)
-			)
-		)
-		(property "Datasheet" "~"
-			(at 262.89 134.62 0)
+			(at 260.35 134.62 0)
+			(effects
+				(font
+					(size 1.27 1.27)
+				)
+				(hide yes)
+			)
+		)
+		(property "Datasheet" "~"
+			(at 260.35 134.62 0)
 			(effects
 				(font
@@
 		)
 		(property "Description" "Fiducial Marker"
-			(at 262.89 134.62 0)
+			(at 260.35 134.62 0)
 			(effects
 				(font
@@
 	(symbol
 		(lib_id "Mechanical:Fiducial")
-		(at 262.89 144.78 0)
+		(at 260.35 144.78 0)
 		(unit 1)
 		(exclude_from_sim no)
@@
 		(fields_autoplaced yes)
 		(property "Reference" "FID6"
-			(at 265.43 143.5099 0)
+			(at 262.89 143.5099 0)
 			(effects
 				(font
@@
 		)
 		(property "Value" "Fiducial"
-			(at 265.43 146.0499 0)
+			(at 262.89 146.0499 0)
 			(effects
 				(font
@@
 		)
 		(property "Footprint" "Fiducial:Fiducial_1.5mm_Mask3mm"
-			(at 262.89 144.78 0)
-			(effects
-				(font
-					(size 1.27 1.27)
-				)
-				(hide yes)
-			)
-		)
-		(property "Datasheet" "~"
-			(at 262.89 144.78 0)
+			(at 260.35 144.78 0)
+			(effects
+				(font
+					(size 1.27 1.27)
+				)
+				(hide yes)
+			)
+		)
+		(property "Datasheet" "~"
+			(at 260.35 144.78 0)
 			(effects
 				(font
@@
 		)
 		(property "Description" "Fiducial Marker"
-			(at 262.89 144.78 0)
+			(at 260.35 144.78 0)
 			(effects
 				(font
@@
 	(symbol
 		(lib_id "Mechanical:Fiducial")
-		(at 262.89 139.7 0)
+		(at 260.35 139.7 0)
 		(unit 1)
 		(exclude_from_sim no)
@@
 		(fields_autoplaced yes)
 		(property "Reference" "FID5"
-			(at 265.43 138.4299 0)
+			(at 262.89 138.4299 0)
 			(effects
 				(font
@@
 		)
 		(property "Value" "Fiducial"
-			(at 265.43 140.9699 0)
+			(at 262.89 140.9699 0)
 			(effects
 				(font
@@
 		)
 		(property "Footprint" "Fiducial:Fiducial_1.5mm_Mask3mm"
-			(at 262.89 139.7 0)
-			(effects
-				(font
-					(size 1.27 1.27)
-				)
-				(hide yes)
-			)
-		)
-		(property "Datasheet" "~"
-			(at 262.89 139.7 0)
+			(at 260.35 139.7 0)
+			(effects
+				(font
+					(size 1.27 1.27)
+				)
+				(hide yes)
+			)
+		)
+		(property "Datasheet" "~"
+			(at 260.35 139.7 0)
 			(effects
 				(font
@@
 		)
 		(property "Description" "Fiducial Marker"
-			(at 262.89 139.7 0)
+			(at 260.35 139.7 0)
 			(effects
 				(font
@@
 	(symbol
 		(lib_id "Mechanical:Fiducial")
-		(at 224.79 134.62 0)
+		(at 223.52 134.62 0)
 		(unit 1)
 		(exclude_from_sim no)
@@
 		(fields_autoplaced yes)
 		(property "Reference" "FID1"
-			(at 227.33 133.3499 0)
+			(at 226.06 133.3499 0)
 			(effects
 				(font
@@
 		)
 		(property "Value" "Fiducial"
-			(at 227.33 135.8899 0)
+			(at 226.06 135.8899 0)
 			(effects
 				(font
@@
 		)
 		(property "Footprint" "Fiducial:Fiducial_1.5mm_Mask3mm"
-			(at 224.79 134.62 0)
-			(effects
-				(font
-					(size 1.27 1.27)
-				)
-				(hide yes)
-			)
-		)
-		(property "Datasheet" "~"
-			(at 224.79 134.62 0)
+			(at 223.52 134.62 0)
+			(effects
+				(font
+					(size 1.27 1.27)
+				)
+				(hide yes)
+			)
+		)
+		(property "Datasheet" "~"
+			(at 223.52 134.62 0)
 			(effects
 				(font
@@
 		)
 		(property "Description" "Fiducial Marker"
-			(at 224.79 134.62 0)
-			(effects
-				(font
+			(at 223.52 134.62 0)
+			(effects
+				(font
