File: OPEN_WEIGHT.kicad_pcb (KiCad board)
At the start: 4 copper layers, 54 x 48 mm, 78 parts, among them IC2 TPS61086DRCR, J1 Conn_01x07_Pin, J2 21033213501, J4 21033213501, Q1 SI2303CDS-T1-GE3, U1 AD7190WBRUZ, U2 LT3042IMSE, Y2 CSTCR4M91G53-R0

Commit message: Clean up project for KDT template: rename, metadata, KiCad 10 CI
- Rename project Cellule_de_force_V2 -> OPEN_WEIGHT and sheets after their function
  (fix AD7910 -> AD7190 typo), update all sheet/project references in sch/pcb/pro
- Real title-block titles, sheet headers use ${TITLE}, restore KDT drawing sheets,
  remove template leftovers from PCB title block
- kibot_main.yaml: COMPANY = OPEN THRUST LAB, GIT_URL = foukouda/OPEN_WEIGHT
- CI: add KiCad 10 (KiBot v2_dk10), PRELIMINARY variant on dev
- README now generated from kibot_resources/templates/readme.txt; fill CHANGELOG
- Move mechanical CAD to Mechanical/, extend .gitignore, untrack 3Dx logs

Co-Authored-By: Claude Opus 5.5 <noreply@anthropic.com>
Connections:
- net /Project Architecture/AD7910_Weight_sensor/IN-OUT+ renamed /Project Architecture/AD7190_Weight_Sensor/IN-OUT+
- net /Project Architecture/AD7910_Weight_sensor/IN-OUT+2 renamed /Project Architecture/AD7190_Weight_Sensor/IN-OUT+2
- net /Project Architecture/AD7910_Weight_sensor/IN-OUT- renamed /Project Architecture/AD7190_Weight_Sensor/IN-OUT-
- net /Project Architecture/AD7910_Weight_sensor/IN-OUT-2 renamed /Project Architecture/AD7190_Weight_Sensor/IN-OUT-2
- net /Project Architecture/Connecteur/IN-OUT+2 renamed /Project Architecture/Connectors/IN-OUT+2
- net /Project Architecture/Connecteur/IN-OUT-2 renamed /Project Architecture/Connectors/IN-OUT-2
- net /Project Architecture/LT3042_6V_5VA/PG renamed /Project Architecture/LT3042_6V_to_5VA/PG
- net /Project Architecture/LT3042_6V_5VA/PGFB renamed /Project Architecture/LT3042_6V_to_5VA/PGFB
- net /Project Architecture/LT3042_6V_5VA/SET renamed /Project Architecture/LT3042_6V_to_5VA/SET

Commit message: Fix load-cell connectivity between Connectors and AD7190 sheets
IN-OUT/IN-SENSE were local labels on two sheets, so the connectors were not
connected to the ADC in the schematic. Convert them to global labels (IN-SENSE
merged into SENSE), and align label polarity on J2/J4 with the routed copper.

Co-Authored-By: Claude Opus 5.5 <noreply@anthropic.com>
Connections:
- J2 pad 1: /Project Architecture/Connectors/IN-OUT+2 -> IN-OUT+2
- J2 pad 2: /Project Architecture/Connectors/IN-OUT-2 -> IN-OUT-2
- R1 pad 1: /Project Architecture/AD7190_Weight_Sensor/IN-OUT+2 -> IN-OUT-2
- R2 pad 1: /Project Architecture/AD7190_Weight_Sensor/IN-OUT-2 -> IN-OUT+2
- R4 pad 1: /Project Architecture/AD7190_Weight_Sensor/IN-OUT+ -> IN-OUT+
- R5 pad 1: /Project Architecture/AD7190_Weight_Sensor/IN-OUT- -> IN-OUT-
Routing:
- net IN-OUT+2: track 0.00 -> 10.1 mm
- net /Project Architecture/Connectors/IN-OUT+2: track 10.1 -> 0.00 mm
- net IN-OUT-2: track 0.00 -> 7.51 mm
- net /Project Architecture/Connectors/IN-OUT-2: track 7.51 -> 0.00 mm
Changed lines of the file:
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@@
 			(layers "F.Cu" "F.Mask" "F.Paste")
 			(roundrect_rratio 0.25)
-			(net "/Project Architecture/AD7190_Weight_Sensor/IN-OUT-2")
+			(net "IN-OUT+2")
 			(pintype "passive")
 		)
@@
 			(layers "F.Cu" "F.Mask" "F.Paste")
 			(roundrect_rratio 0.25)
-			(net "/Project Architecture/AD7190_Weight_Sensor/IN-OUT+")
+			(net "IN-OUT+")
 			(pintype "passive")
 		)
@@
 			(layers "F.Cu" "F.Mask" "F.Paste")
 			(roundrect_rratio 0.25)
-			(net "/Project Architecture/AD7190_Weight_Sensor/IN-OUT+2")
+			(net "IN-OUT-2")
 			(pintype "passive")
 		)
@@
 			(layers "*.Cu" "*.Mask")
 			(remove_unused_layers no)
-			(net "/Project Architecture/Connectors/IN-OUT+2")
+			(net "IN-OUT+2")
 			(pinfunction "1")
 			(pintype "passive")
@@
 			(layers "*.Cu" "*.Mask")
 			(remove_unused_layers no)
-			(net "/Project Architecture/Connectors/IN-OUT-2")
+			(net "IN-OUT-2")
 			(pinfunction "2")
 			(pintype "passive")
@@
 			(layers "F.Cu" "F.Mask" "F.Paste")
 			(roundrect_rratio 0.25)
-			(net "/Project Architecture/AD7190_Weight_Sensor/IN-OUT-")
+			(net "IN-OUT-")
 			(pintype "passive")
 		)
@@
 		(width 0.2)
 		(layer "F.Cu")
-		(net "/Project Architecture/Connectors/IN-OUT+2")
+		(net "IN-OUT+2")
 	)
 	(segment
@@
 		(width 0.2)
 		(layer "F.Cu")
-		(net "/Project Architecture/Connectors/IN-OUT+2")
+		(net "IN-OUT+2")
 	)
 	(segment
@@
 		(width 0.2)
 		(layer "F.Cu")
-		(net "/Project Architecture/Connectors/IN-OUT+2")
+		(net "IN-OUT+2")
 	)
 	(arc
@@
 		(width 0.2)
 		(layer "F.Cu")
-		(net "/Project Architecture/Connectors/IN-OUT+2")
+		(net "IN-OUT+2")
 	)
 	(arc
@@
 		(width 0.2)
 		(layer "F.Cu")
-		(net "/Project Architecture/Connectors/IN-OUT+2")
+		(net "IN-OUT+2")
 	)
 	(arc
@@
 		(width 0.2)
 		(layer "F.Cu")
-		(net "/Project Architecture/Connectors/IN-OUT+2")
+		(net "IN-OUT+2")
 	)
 	(arc
@@
 		(width 0.2)
 		(layer "F.Cu")
-		(net "/Project Architecture/Connectors/IN-OUT+2")
+		(net "IN-OUT+2")
 	)
 	(segment
@@
 		(width 0.2)
 		(layer "F.Cu")
-		(net "/Project Architecture/Connectors/IN-OUT-2")
+		(net "IN-OUT-2")
 	)
 	(segment
@@
 		(width 0.2)
 		(layer "F.Cu")
-		(net "/Project Architecture/Connectors/IN-OUT-2")
+		(net "IN-OUT-2")
 	)
 	(segment
@@
 		(width 0.2)
 		(layer "F.Cu")
-		(net "/Project Architecture/Connectors/IN-OUT-2")
+		(net "IN-OUT-2")
 	)
 	(segment
@@
 		(width 0.2)
 		(layer "F.Cu")
-		(net "/Project Architecture/Connectors/IN-OUT-2")
+		(net "IN-OUT-2")
 	)
 	(arc
@@
 		(width 0.2)
 		(layer "F.Cu")
-		(net "/Project Architecture/Connectors/IN-OUT-2")
+		(net "IN-OUT-2")
 	)
 	(arc
@@
 		(width 0.2)
 		(layer "F.Cu")
-		(net "/Project Architecture/Connectors/IN-OUT-2")
+		(net "IN-OUT-2")
 	)
 	(arc
@@
 		(width 0.2)
 		(layer "F.Cu")
-		(net "/Project Architecture/Connectors/IN-OUT-2")
+		(net "IN-OUT-2")
 	)
 	(segment

Commit message: Self-contained libraries, JLCPCB rules, ERC/DRC cleanup
- lib/: project symbol library (19 symbols), footprint library (17 footprints)
  and all 3D models (15), referenced through ${KIPRJMOD} + project lib tables.
  A fresh clone now opens with every symbol, footprint and 3D model.
- Remove duplicated / absolute 3D model paths (C:/Users/..., ${KICAD_FOOTPRINT})
- OPEN_WEIGHT.kicad_dru: JLCPCB 4-layer rules; stackup JLC04161H-7628; board minimums
- AD7190 footprint: drop per-pad 0.102 mm mask margin (mask bridges at 0.65 mm pitch)
- Exclude unplaced TP/FID symbols from board; PWR_FLAGs; decorative wires -> lines
- Local text variables in .kicad_pro; Revision History wired to [Unreleased]
- get_changelog.py: accept "## [Unreleased]" without date
ERC: 0 errors. DRC: 0 errors except 10 courtyard overlaps (placement), 0 parity issues.

Co-Authored-By: Claude Opus 5.5 <noreply@anthropic.com>
Parts:
- C1, C10, C11, C12, C13, C15, C16, C17, C18, C19, C2, C20, C21, C22, C23, C24, C25, C26, C27, C28, C29, C3, C4, C5, C6, C7, C8, C9: footprint Capacitor_SMD:C_0603_1608Metric -> OPEN_WEIGHT:C_0603_1608Metric
- C14: footprint TAJA225K016RNJ:CAPPM3216X180N -> OPEN_WEIGHT:CAPPM3216X180N
- D1, D2, D4: footprint LED_SMD:LED_0603_1608Metric -> OPEN_WEIGHT:LED_0603_1608Metric
- D3: footprint Diode_SMD:D_SOD-123F -> OPEN_WEIGHT:D_SOD-123F
- H1, H2, H3, H4: footprint MountingHole:MountingHole_3.2mm_M3_Pad_Via -> OPEN_WEIGHT:MountingHole_3.2mm_M3_Pad_Via
- H5: footprint WE-SHC_THT-FRAME:WE-SHC_THT-FRAME_36503205 -> OPEN_WEIGHT:WE-SHC_THT-FRAME_36503205
- IC2: footprint TPS61086DRCR:TPS16412DRCR -> OPEN_WEIGHT:TPS16412DRCR
- J1: footprint Connector_JST:JST_XH_B7B-XH-AM_1x07_P2.50mm_Vertical -> OPEN_WEIGHT:JST_XH_B7B-XH-AM_1x07_P2.50mm_Vertical
- J2, J4: footprint 21033213501:21033213501 -> OPEN_WEIGHT:21033213501
- L1: footprint 7447785004:7447785004 -> OPEN_WEIGHT:7447785004
- Q1: footprint Package_TO_SOT_SMD:SOT-23-3 -> OPEN_WEIGHT:SOT-23-3
- R1, R10, R11, R12, R13, R14, R15, R16, R17, R18, R2, R3, R4, R5, R6, R8, R9: footprint Resistor_SMD:R_0603_1608Metric -> OPEN_WEIGHT:R_0603_1608Metric
- RN1: footprint Resistor_SMD:R_Array_Concave_4x0603 -> OPEN_WEIGHT:R_Array_Concave_4x0603
- TP11, TP12, TP13, TP14, TP15, TP16, TP17, TP18, TP2, TP4, TP5: footprint TestPoint:TestPoint_Pad_D1.5mm -> OPEN_WEIGHT:TestPoint_Pad_D1.5mm
- U1: footprint AD7190WBRUZ:SOP65P640X120-24N -> OPEN_WEIGHT:SOP65P640X120-24N
- U2: footprint Package_SO:MSOP-10-1EP_3x3mm_P0.5mm_EP2.2x3.1mm_Mask1.83x1.89mm_ThermalVias -> OPEN_WEIGHT:MSOP-10-1EP_3x3mm_P0.5mm_EP2.2x3.1mm_Mask1.83x1.89mm_ThermalVias
- Y2: footprint CSTCR4M91G53-R0:OSC_CSTCR4M91G53-R0 -> OPEN_WEIGHT:OSC_CSTCR4M91G53-R0
Other:
- rule pad_to_mask_clearance: 0.05 -> 0
