File: OPEN_WEIGHT.kicad_pcb (KiCad board)
At the start: 4 copper layers, 54 x 48 mm, 78 parts, among them IC2 TPS61086DRCR, J1 Conn_01x07_Pin, J2 21033213501, J4 21033213501, Q1 SI2303CDS-T1-GE3, U1 AD7190WBRUZ, U2 LT3042IMSE, Y2 CSTCR4M91G53-R0

Commit message: Restyle the schematic like OPEN_PHASE, merge the power sheets, rework the bottom silkscreen
- Schematic: all sheets on A3 in the OPEN_PHASE look (red header bands,
  DESCRIPTION / DESIGN NOTE / LAYOUT NOTE / CALCULS & BUDGET panels in
  French, TEST POINTS panel, References in the title block)
- Title block: INGENIERIE FRANCE logo in KDT_Template_GIT.kicad_wks,
  per-sheet logo images removed
- Power - Sequencing rebuilt with curves from LTspice simulations 01-04
- TPS61086 and LT3042 sheets merged into Power Supply - Analog Rails
  (page 5, keeps the TPS sheet UUID); pages renumbered to 9, local nets
  renamed to /Project Architecture/Power_Supply/*, PCB links updated
- PCB: per-rail net colours (+3.3V, +6V, +5VA, GND) as on OPEN_PHASE
- PCB B.SilkS: test point pills with Arial Black knockout names, J1
  pinout cells, E+/E-/S+/S- tags on the M12 pads, CELL 1 / CELL 2 titles
  and a LOAD CELL wiring panel

Netlist connectivity, ERC (2 warnings) and copper DRC unchanged;
schematic parity clean.

Co-Authored-By: Claude Opus 5.5 <noreply@anthropic.com>
Connections:
- net /Project Architecture/LT3042_6V_to_5VA/PG renamed /Project Architecture/Power_Supply/PG
- net /Project Architecture/LT3042_6V_to_5VA/PGFB renamed /Project Architecture/Power_Supply/PGFB
- net /Project Architecture/LT3042_6V_to_5VA/SET renamed /Project Architecture/Power_Supply/SET
- net /Project Architecture/TPS61086_3.3V_to_6V/COMP renamed /Project Architecture/Power_Supply/COMP
- net /Project Architecture/TPS61086_3.3V_to_6V/FB renamed /Project Architecture/Power_Supply/FB
- net /Project Architecture/TPS61086_3.3V_to_6V/SS renamed /Project Architecture/Power_Supply/SS
Other:
- board text added: "+6V"
- board text added: "CELL 1"
- board text added: "CELL 2"
- board text added: "E+"
- board text added: "E−"
- board text added: "LOAD CELL"
- board text added: "S+"
- board text added: "S−"
- board text removed: "3.3V"
- board text removed: "5VA"
- board text removed: "6V"
