File: Connectors.kicad_sch (KiCad schematic)
At the start: 4 parts, among them J1 Conn_01x07_Pin, J2 21033213501, J4 21033213501

Commit message: Fill template pages: block diagram, power sequencing, notes, revision history
Block Diagram and Power - Sequencing rebuilt from the real design (values computed
from the schematic); cover-page design notes, connector pinout notes, title-block
references; kicad-mcp-pro MCP config (.mcp.json).

Co-Authored-By: Claude Opus 5.5 <noreply@anthropic.com>
Other:
- note added: "J2/J4 21033213501, H5 WE-SHC"
- note added: "JST XH B7B-XH-AM (J1)"
- note removed: "Flexible I/O source configuration"
- note removed: "Flexible I/O worked examples"
Changed lines of the file:
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@@
 		)
 	)
-	(text "Flexible I/O worked examples"
+	(text "JST XH B7B-XH-AM (J1)"
 		(exclude_from_sim no)
 		(at 265.43 254 0)
@@
 		)
 	)
-	(text "Flexible I/O source configuration"
+	(text "J2/J4 21033213501, H5 WE-SHC"
 		(exclude_from_sim no)
 		(at 265.43 256.54 0)
@@
 		)
 	)
-	(text_box "Block Description"
+	(text_box ""
 		(exclude_from_sim no)
 		(at 46.99 194.31 0)
@@
 		)
 	)
-	(text_box "Block Description"
+	(text_box ""
 		(exclude_from_sim no)
 		(at 140.97 228.6 0)
@@
 		)
 	)
-	(text_box "Block Description"
+	(text_box ""
 		(exclude_from_sim no)
 		(at 46.99 228.6 0)
@@
 		)
 	)
-	(text_box "DESIGN NOTE:\nblabla"
+	(text_box "DESIGN NOTE:\nJ1 host header (JST-XH, 7 pins):\n1 +3.3V   2 CS   3 DIN   4 DOUT/RDY\n5 SYNC   6 SCLK   7 GND"
 		(exclude_from_sim no)
-		(at 77.47 143.51 0)
-		(size 21.59 15.24)
+		(at 52.07 58.42 0)
+		(size 76.2 26)
 		(margins 1.3525 1.3525 1.3525 1.3525)
 		(stroke
@@
 		)
 	)
-	(text_box "Block Description"
+	(text_box ""
 		(exclude_from_sim no)
 		(at 231.14 228.6 0)
@@
 		)
 	)
-	(text_box "LAYOUT NOTE:\nblabla"
+	(text_box "LAYOUT NOTE:\nH5 shielding frame covers the AD7190\nfront-end; connector shells tied to GND."
 		(exclude_from_sim no)
-		(at 101.6 143.51 0)
-		(size 26.67 15.24)
+		(at 52.07 125.73 0)
+		(size 76.2 18)
 		(margins 1.4525 1.4525 1.4525 1.4525)
 		(stroke
@@
 		)
 	)
-	(text_box "Block Description"
+	(text_box "Pinout and notes"
 		(exclude_from_sim no)
 		(at 46.99 156.21 0)
@@
 		)
 	)
-	(text_box "Block Description"
+	(text_box "Host and load-cell connectors"
 		(exclude_from_sim no)
 		(at 142.24 192.405 0)
@@
 		)
 	)
-	(text_box "Block Description"
+	(text_box ""
 		(exclude_from_sim no)
 		(at 318.77 228.6 0)
@@
 		)
 	)
-	(text_box "DESIGN NOTE:\nblabla"
+	(text_box "DESIGN NOTE:\nJ2/J4 load cell (5 pins):\n1 OUT, 2 OUT (signal pair), 3 EXC+ (SENSE+),\n4 EXC- (SENSE-/BPDSW), 5 GND/shield.\nBoth channels read V(pin2) - V(pin1):\nfix the sign in firmware if needed."
 		(exclude_from_sim no)
-		(at 53.34 143.51 0)
-		(size 21.59 15.24)
+		(at 52.07 90.17 0)
+		(size 76.2 30)
 		(margins 1.3525 1.3525 1.3525 1.3525)
 		(stroke
@@
 	(text "Power flags: +3.3V and GND come from the host connector J1,\n+6V from the TPS61086 boost (tells ERC these rails are driven)."
 		(exclude_from_sim no)
-		(at 55.88 101.6 0)
+		(at 55.88 207.01 0)
 		(effects
 			(font
@@
 	(symbol
 		(lib_id "power:+3.3V")
-		(at 63.5 85.09 0)
+		(at 63.5 190.50 0)
 		(unit 1)
 		(body_style 1)
@@
 		(dnp no)
 		(property "Reference" "#PWR10"
-			(at 63.5 85.09 0)
+			(at 63.5 190.50 0)
 			(hide yes)
 			(show_name no)
@@
 		)
 		(property "Value" "+3.3V"
-			(at 63.5 81.28 0)
+			(at 63.5 186.69 0)
 			(show_name no)
 			(do_not_autoplace no)
@@
 		)
 		(property "Footprint" ""
-			(at 63.5 85.09 0)
+			(at 63.5 190.50 0)
 			(hide yes)
 			(show_name no)
@@
 		)
 		(property "Datasheet" "~"
-			(at 63.5 85.09 0)
+			(at 63.5 190.50 0)
 			(hide yes)
 			(show_name no)
@@
 		)
 		(property "Description" "Power symbol creates a global label with name \"+3.3V\""
-			(at 63.5 85.09 0)
+			(at 63.5 190.50 0)
 			(hide yes)
 			(show_name no)
@@
 	(symbol
 		(lib_id "power:PWR_FLAG")
-		(at 63.5 85.09 180)
+		(at 63.5 190.50 180)
 		(unit 1)
 		(body_style 1)
@@
 		(dnp no)
 		(property "Reference" "#FLG01"
-			(at 63.5 85.09 0)
+			(at 63.5 190.50 0)
 			(hide yes)
 			(show_name no)
@@
 		)
 		(property "Value" "PWR_FLAG"
-			(at 63.5 90.17 0)
+			(at 63.5 195.58 0)
 			(show_name no)
 			(do_not_autoplace no)
@@
 		)
 		(property "Footprint" ""
-			(at 63.5 85.09 0)
+			(at 63.5 190.50 0)
 			(hide yes)
 			(show_name no)
@@
 		)
 		(property "Datasheet" "~"
-			(at 63.5 85.09 0)
+			(at 63.5 190.50 0)
 			(hide yes)
 			(show_name no)
@@
 		)
 		(property "Description" "Special symbol for telling ERC where power comes from"
-			(at 63.5 85.09 0)
+			(at 63.5 190.50 0)
 			(hide yes)
 			(show_name no)
@@
 	(symbol
 		(lib_id "power:GND")
-		(at 104.14 85.09 0)
+		(at 104.14 190.50 0)
 		(unit 1)
 		(body_style 1)
@@
 		(dnp no)
 		(property "Reference" "#PWR12"
-			(at 104.14 85.09 0)
+			(at 104.14 190.50 0)
 			(hide yes)
 			(show_name no)
@@
 		)
 		(property "Value" "GND"
-			(at 104.14 90.17 0)
+			(at 104.14 195.58 0)
 			(show_name no)
 			(do_not_autoplace no)
@@
 		)
 		(property "Footprint" ""
-			(at 104.14 85.09 0)
+			(at 104.14 190.50 0)
 			(hide yes)
 			(show_name no)
@@
 		)
 		(property "Datasheet" "~"
-			(at 104.14 85.09 0)
+			(at 104.14 190.50 0)
 			(hide yes)
 			(show_name no)
@@
 		)
 		(property "Description" "Power symbol creates a global label with name \"GND\""
-			(at 104.14 85.09 0)
+			(at 104.14 190.50 0)
 			(hide yes)
 			(show_name no)
@@
 	(symbol
 		(lib_id "power:PWR_FLAG")
-		(at 104.14 85.09 0)
+		(at 104.14 190.50 0)
 		(unit 1)
 		(body_style 1)
@@
 		(dnp no)
 		(property "Reference" "#FLG03"
-			(at 104.14 85.09 0)
+			(at 104.14 190.50 0)
 			(hide yes)
 			(show_name no)
@@
 		)
 		(property "Value" "PWR_FLAG"
-			(at 104.14 80.01 0)
+			(at 104.14 185.42 0)
 			(show_name no)
 			(do_not_autoplace no)
@@
 		)
 		(property "Footprint" ""
-			(at 104.14 85.09 0)
+			(at 104.14 190.50 0)
 			(hide yes)
 			(show_name no)
@@
 		)
 		(property "Datasheet" "~"
-			(at 104.14 85.09 0)
+			(at 104.14 190.50 0)
 			(hide yes)
 			(show_name no)
@@
 		)
 		(property "Description" "Special symbol for telling ERC where power comes from"
-			(at 104.14 85.09 0)
+			(at 104.14 190.50 0)
 			(hide yes)
 			(show_name no)
