File: OPEN_WEIGHT.kicad_sch (KiCad schematic)
At the start: 0 parts

Commit message: Clean up project for KDT template: rename, metadata, KiCad 10 CI
- Rename project Cellule_de_force_V2 -> OPEN_WEIGHT and sheets after their function
  (fix AD7910 -> AD7190 typo), update all sheet/project references in sch/pcb/pro
- Real title-block titles, sheet headers use ${TITLE}, restore KDT drawing sheets,
  remove template leftovers from PCB title block
- kibot_main.yaml: COMPANY = OPEN THRUST LAB, GIT_URL = foukouda/OPEN_WEIGHT
- CI: add KiCad 10 (KiBot v2_dk10), PRELIMINARY variant on dev
- README now generated from kibot_resources/templates/readme.txt; fill CHANGELOG
- Move mechanical CAD to Mechanical/, extend .gitignore, untrack 3Dx logs

Co-Authored-By: Claude Opus 5.5 <noreply@anthropic.com>
Other:
- title: (none) -> OPEN_WEIGHT - AD7190
Changed lines of the file:
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@@
 	(paper "A3")
 	(title_block
+		(title "OPEN_WEIGHT - AD7190")
 		(date "2025-01-12")
 		(rev "${REVISION}")
@@
 		)
 		(instances
-			(project "Cellule_de_force_V2"
+			(project "OPEN_WEIGHT"
 				(path "/f9e05184-c88b-4a88-ae9c-ab2bdb32be7c"
 					(reference "#SYM1")
@@
 		)
 		(instances
-			(project "Cellule_de_force_V2"
+			(project "OPEN_WEIGHT"
 				(path "/f9e05184-c88b-4a88-ae9c-ab2bdb32be7c"
 					(page "9")
@@
 		)
 		(instances
-			(project "Cellule_de_force_V2"
+			(project "OPEN_WEIGHT"
 				(path "/f9e05184-c88b-4a88-ae9c-ab2bdb32be7c"
 					(page "10")
@@
 		)
 		(instances
-			(project "Cellule_de_force_V2"
+			(project "OPEN_WEIGHT"
 				(path "/f9e05184-c88b-4a88-ae9c-ab2bdb32be7c"
 					(page "2")
@@
 		)
 		(instances
-			(project "Cellule_de_force_V2"
+			(project "OPEN_WEIGHT"
 				(path "/f9e05184-c88b-4a88-ae9c-ab2bdb32be7c"
 					(page "3")

Commit message: Fill template pages: block diagram, power sequencing, notes, revision history
Block Diagram and Power - Sequencing rebuilt from the real design (values computed
from the schematic); cover-page design notes, connector pinout notes, title-block
references; kicad-mcp-pro MCP config (.mcp.json).

Co-Authored-By: Claude Opus 5.5 <noreply@anthropic.com>
Other:
- note added: "OPEN_WEIGHT - AD7190 24-bit load-cell front-end, part of OPEN THRUST LAB. Single +3.3 V host supply, SPI interface, 2 x 4-wire bridge inputs."
- note removed: "Comment"
Changed lines of the file:
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@@
 		)
 	)
-	(text "Comment"
+	(text "OPEN_WEIGHT - AD7190 24-bit load-cell front-end, part of OPEN THRUST LAB.\nSingle +3.3 V host supply, SPI interface, 2 x 4-wire bridge inputs."
 		(exclude_from_sim no)
 		(at 222.25 177.8 0)
@@
 		)
 	)
-	(text_box "DESIGN NOTE:\nExample text for cautionary design notes."
+	(text_box "DESIGN NOTE:\nSPI mode 3,\nSCLK <= 5 MHz,\nRDY on DOUT."
 		(exclude_from_sim no)
 		(at 96.52 258.445 0)
@@
 		)
 	)
-	(text_box "DESIGN NOTE:\nExample text for debug notes."
+	(text_box "DEBUG NOTE:\nTP on every rail.\nWait >= 600 ms (PG)\nbefore ADC init."
 		(exclude_from_sim no)
 		(at 61.595 258.445 0)
@@
 		)
 	)
-	(text_box "DESIGN NOTE:\nExample text for critical design notes."
+	(text_box "DESIGN NOTE:\nREFIN1 = bridge\nexcitation:\nratiometric."
 		(exclude_from_sim no)
 		(at 131.445 258.445 0)
@@
 		)
 	)
-	(text_box "LAYOUT NOTE:\nExample text for critical layout guidelines."
+	(text_box "LAYOUT NOTE:\nAFE under the\nWE-SHC shield H5,\nboost SW node away."
 		(exclude_from_sim no)
 		(at 166.37 258.445 0)
@@
 		)
 	)
-	(text_box "DESIGN NOTE:\nExample text for informational design notes."
+	(text_box "DESIGN NOTE:\n+3.3V host -> TPS61086\n6 V -> LT3042 +5VA\n(AVDD + excitation)"
 		(exclude_from_sim no)
 		(at 26.67 258.445 0)
